File: test_boards/10CL006YE144C8G/10CL006YE144C8G.kicad_sch (KiCad schematic)
At the start: 81 parts, among them IC1 10CL006YE144C8G, J1 CL_JTAG, U1 W25Q128JVS, Y1 SG-7050CAN

Commit message: Правки kicad проекта
Parts:
- C27: value 4.7 uF -> 100 nF
Changed lines of the file:
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@@
 			)
 		)
-		(property "Value" "4.7 uF"
+		(property "Value" "100 nF"
 			(at 52.07 226.06 90)
 			(show_name no)

Commit message: добавлен автоматический генератор номиналов для конфига
Parts:
- added C37: 4.7 uF, Capacitor_SMD:C_0603_1608Metric_Pad1.08x0.95mm_HandSolder, symbol Device:C
- renumbered C37 to C38, C38 to C39, C39 to C40, C40 to C41, C41 to C42, C42 to C43, C43 to C44, C44 to C45, C45 to C46, C46 to C47, C47 to C48, C48 to C49, C49 to C50, C50 to C51, C51 to C52, C52 to C53, C53 to C54, C54 to C55, C55 to C56, C56 to C57, C57 to C58, C58 to C59, C59 to C60, C60 to C61, C61 to C62
Connections:
- net +3V3_VCCIO: now also C37.1
- net GND: now also C37.2
