File: test_boards/10CL006YE144C8G/10CL006YE144C8G.kicad_sch (KiCad schematic)
At the start: 83 parts, among them IC1 10CL006YE144C8G, J1 CL_JTAG, U1 W25Q128JVS, Y1 SG-7050CAN

Commit message: Перешёл на шаблоны. Шаблоны спиц уже расставляются по местам
Parts:
- removed C55: 4.7 uF, Capacitor_SMD:C_0603_1608Metric_Pad1.08x0.95mm_HandSolder, symbol Device:C
- added C15, C16: 100 nF, Capacitor_SMD:C_0402_1005Metric_Pad0.74x0.62mm_HandSolder, symbol Device:C
- added C29, C30, C31, C32, C40, C41: 4.7 uF, Capacitor_SMD:C_0603_1608Metric_Pad1.08x0.95mm_HandSolder, symbol Device:C
- C21: renamed from C30; TemplateRole (none) -> VCCIO1_LIGHT
- C5: TemplateRole (none) -> VCCIO1_HEAVY
- renumbered C15 to C17, C16 to C18, C17 to C19, C18 to C20, C31 to C22, C32 to C23, C33 to C24, C34 to C25, C35 to C26, C36 to C27, C37 to C28, C40 to C33, C41 to C34, C42 to C35, C43 to C36, C44 to C37, C45 to C38, C46 to C39, C19 to C42, C20 to C43, C21 to C44, C22 to C45, C23 to C46, C24 to C47, C25 to C48, C26 to C49, C27 to C50, C47 to C51, C48 to C52, C49 to C53, C50 to C54, C53 to C55, C54 to C56, C38 to C57, C39 to C58, C28 to C59, C29 to C60, C51 to C61, C52 to C62, C56 to C63, C57 to C64, C59 to C65, C58 to C66, C61 to C67, C60 to C68, C62 to C69, C63 to C70, R4 to R2, R5 to R4, R6 to R5, R2 to R6
Connections:
- net +1V2_VCCINT: now also C40.1, C41.1
- net +3V3_VCCIO: now also C15.1, C16.1, C29.1, C30.1, C31.1, C32.1
- net GND: now also C15.2, C16.2, C29.2, C30.2, C31.2, C32.2, C40.2, C41.2
Other:
- moved on the sheet: C1, C10, C11, C12, C13, C17, C18, C19, C2, C20, C21, C22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
