File: test_boards/10CL006YE144C8G/10CL006YE144C8G.kicad_sch (KiCad schematic)
At the start: 88 parts, among them IC1 10CL006YE144C8G, J1 CL_JTAG, U1 W25Q128JVS, Y1 SG-7050CAN

Commit message: Добавлен скрипт диагностиги падения KiCad
Parts:
- C1, C2, C3, C4: Role (none) -> PI_FILTER_C1
- C17, C18, C19: Role LIGHT -> PI_FILTER_C2
- C20: Role LIGHT -> PI_FILTER_C2; TemplateRole LIGHT -> (none)
- C49, C50, C51, C52: Role (none) -> PI_FILTER_C3
- FB1, FB2, FB3, FB4: Role (none) -> PI_FILTER_FB
Changed lines of the file:
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@@
 			)
 		)
-		(property "Role" "LIGHT"
+		(property "Role" "PI_FILTER_C2"
 			(at 44.45 52.07 0)
 			(hide yes)
@@
 			)
 		)
-		(property "Role" "LIGHT"
+		(property "Role" "PI_FILTER_C2"
 			(at 44.45 30.48 0)
 			(hide yes)
@@
 			)
 		)
+		(property "Role" "PI_FILTER_C1"
+			(at 34.29 30.48 0)
+			(hide yes)
+			(show_name no)
+			(do_not_autoplace no)
+			(effects
+				(font
+					(size 1.27 1.27)
+				)
+			)
+		)
 		(pin "2"
 		)
@@
 			)
 		)
+		(property "Role" "PI_FILTER_C1"
+			(at 0 0 0)
+			(show_name no)
+			(do_not_autoplace no)
+			(effects
+				(font
+					(size 1.27 1.27)
+				)
+			)
+		)
 		(pin "2"
 		)
@@
 			)
 		)
+		(property "Role" "PI_FILTER_C1"
+			(at 0 0 0)
+			(show_name no)
+			(do_not_autoplace no)
+			(effects
+				(font
+					(size 1.27 1.27)
+				)
+			)
+		)
 		(pin "2"
 		)
@@
 			)
 		)
+		(property "Role" "PI_FILTER_C1"
+			(at 34.29 102.87 0)
+			(hide yes)
+			(show_name no)
+			(do_not_autoplace no)
+			(effects
+				(font
+					(size 1.27 1.27)
+				)
+			)
+		)
 		(pin "2"
 		)
@@
 			)
 		)
+		(property "Role" "PI_FILTER_C3"
+			(at 85.09 102.87 0)
+			(hide yes)
+			(show_name no)
+			(do_not_autoplace no)
+			(effects
+				(font
+					(size 1.27 1.27)
+				)
+			)
+		)
 		(pin "2"
 		)
@@
 			)
 		)
-		(property "Role" "LIGHT"
+		(property "Role" "PI_FILTER_C2"
 			(at 44.45 77.47 0)
 			(hide yes)
@@
 			)
 		)
-		(property "TemplateRole" "LIGHT"
-			(at 44.45 102.87 0)
-			(hide yes)
-			(show_name no)
-			(do_not_autoplace no)
-			(effects
-				(font
-					(size 1.27 1.27)
-				)
-			)
-		)
-		(property "Role" "LIGHT"
+		(property "Role" "PI_FILTER_C2"
 			(at 44.45 102.87 0)
 			(hide yes)
@@
 			)
 		)
+		(property "Role" "PI_FILTER_FB"
+			(at 58.42 99.06 0)
+			(hide yes)
+			(show_name no)
+			(do_not_autoplace no)
+			(effects
+				(font
+					(size 1.27 1.27)
+				)
+			)
+		)
 		(pin "1"
 		)
@@
 			)
 		)
+		(property "Role" "PI_FILTER_FB"
+			(at 10.16 106.68 0)
+			(show_name no)
+			(do_not_autoplace no)
+			(effects
+				(font
+					(size 1.27 1.27)
+				)
+			)
+		)
 		(pin "1"
 		)
@@
 			)
 		)
+		(property "Role" "PI_FILTER_FB"
+			(at 58.42 26.67 0)
+			(hide yes)
+			(show_name no)
+			(do_not_autoplace no)
+			(effects
+				(font
+					(size 1.27 1.27)
+				)
+			)
+		)
 		(pin "1"
 		)
@@
 			)
 		)
+		(property "Role" "PI_FILTER_C3"
+			(at 0 0 0)
+			(show_name no)
+			(do_not_autoplace no)
+			(effects
+				(font
+					(size 1.27 1.27)
+				)
+			)
+		)
 		(pin "2"
 		)
@@
 			)
 		)
+		(property "Role" "PI_FILTER_C3"
+			(at 85.09 30.48 0)
+			(hide yes)
+			(show_name no)
+			(do_not_autoplace no)
+			(effects
+				(font
+					(size 1.27 1.27)
+				)
+			)
+		)
 		(pin "2"
 		)
@@
 			)
 		)
+		(property "Role" "PI_FILTER_FB"
+			(at -15.24 132.08 0)
+			(show_name no)
+			(do_not_autoplace no)
+			(effects
+				(font
+					(size 1.27 1.27)
+				)
+			)
+		)
 		(pin "1"
 		)
@@
 			(show_name no)
 			(do_not_autoplace no)
+			(effects
+				(font
+					(size 1.27 1.27)
+				)
+			)
+		)
+		(property "Role" "PI_FILTER_C3"
+			(at 0 0 0)
+			(show_name no)
+			(do_not_autoplace no)

Commit message: добавлено извлечение шаблона с 0 относительно via. Поправил регистр действий. Теперь ищутся реальные компоненты на плате
Parts:
- added C55, C56, C57, C58: 100 nF, Capacitor_SMD:C_0402_1005Metric_Pad0.74x0.62mm_HandSolder, symbol Device:C
- renumbered C55 to C59, C56 to C60, C57 to C61, C58 to C62, C59 to C63, C60 to C64, C61 to C65, C62 to C66, C63 to C67, C64 to C68, C65 to C69, C66 to C70, C67 to C71, C68 to C72
Connections:
- net +1V2_VCCD_PLL: now also C55.1
- net +1V2_VCCINT: now also C56.1
- net +2V5_VCCA: now also C57.1
- net +3V3_VCCIO: now also C58.1
- net GND: now also C55.2, C56.2, C57.2, C58.2
