File: test_boards/10CL006YE144C8G/10CL006YE144C8G.kicad_pcb (KiCad board)
At the start: 2 copper layers, 81 parts, among them IC1 10CL006YE144C8G, J1 CL_JTAG, U1 W25Q128JVS, Y1 SG-7050CAN

Commit message: Правки
Parts:
- added C62: 100 nF, Capacitor_SMD:C_0402_1005Metric_Pad0.74x0.62mm_HandSolder, F.Cu at (108.7, 94.1)
- C27: value 4.7 uF -> 100 nF
- C37: value 100 nF -> 4.7 uF; footprint Capacitor_SMD:C_0402_1005Metric_Pad0.74x0.62mm_HandSolder -> Capacitor_SMD:C_0603_1608Metric_Pad1.08x0.95mm_HandSolder
- C39: value 4.7 uF -> 100 nF; footprint Capacitor_SMD:C_0603_1608Metric_Pad1.08x0.95mm_HandSolder -> Capacitor_SMD:C_0402_1005Metric_Pad0.74x0.62mm_HandSolder
- C46, C54: value 1uF -> 4.7 uF
- C50: value 4.7 uF -> 1uF
- C55, C58, C61: value 100 nF -> 1uF; footprint Capacitor_SMD:C_0402_1005Metric_Pad0.74x0.62mm_HandSolder -> Capacitor_SMD:C_0603_1608Metric_Pad1.08x0.95mm_HandSolder
- C56, C60: value 1uF -> 100 nF; footprint Capacitor_SMD:C_0603_1608Metric_Pad1.08x0.95mm_HandSolder -> Capacitor_SMD:C_0402_1005Metric_Pad0.74x0.62mm_HandSolder
- moved J1 121.0 mm to (90.7, 89.4)
- moved IC1 113.4 mm to (51.6, 71.0)
- moved U1 107.9 mm to (115.5, 94.7)
- moved C10 104.4 mm to (99.0, 94.1)
- moved C11 104.4 mm to (99.0, 96.0)
- moved C12 104.4 mm to (99.0, 98.0)
- moved C21 104.4 mm to (105.5, 84.2)
- moved C22 104.4 mm to (105.5, 86.2)
- moved C23 104.4 mm to (105.5, 88.2)
- moved C24 104.4 mm to (105.5, 90.1)
- moved C25 104.4 mm to (105.5, 92.1)
- moved C26 104.4 mm to (105.5, 94.1)
- moved C28 104.4 mm to (105.5, 96.0)
- moved C29 104.4 mm to (105.5, 98.0)
- moved C5 104.4 mm to (99.0, 84.2)
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Connections:
- C37 pad 1: +1V2_VCCD_PLL -> +3V3_VCCIO
- C39 pad 1: +1V2_VCCINT -> +1V2_VCCD_PLL
- C47 pad 1: +1V2_VCCD_PLL -> +1V2_VCCINT
- C48 pad 1: +2V5_VCCA -> +1V2_VCCD_PLL
- C49 pad 1: +3V3_VCCIO -> +2V5_VCCA
- C50 pad 1: +2V5_VCCA -> +3V3_VCCIO
- C52 pad 1: +1V2_VCCD_PLL -> +2V5_VCCA
- C54 pad 1: +3V3 -> +1V2_VCCD_PLL
- C56 pad 1: +3V3_OSCILL -> +3V3
- C57 pad 1: +3V3 -> +3V3_OSCILL
- C58 pad 1: GND -> +3V3
- C58 pad 2: +3V3_OSCILL -> GND
- C59 pad 1: +3V3 -> GND
- C59 pad 2: GND -> +3V3_OSCILL
- C60 pad 1: +3V3_FLASH -> +3V3
- C61 pad 1: GND -> +3V3_FLASH
- C61 pad 2: +3V3_FLASH -> GND

Commit message: заработала расстановка конденсаторов по радиусу
Parts:
- moved C5 11.1 mm to (91.3, 76.4)
- moved C6 10.2 mm to (91.3, 79.6)
Changed lines of the file:
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@@
 	(footprint "Capacitor_SMD:C_0402_1005Metric_Pad0.74x0.62mm_HandSolder"
 		(layer "F.Cu")
-		(at 99.035 86.195)
+		(at 91.2575 79.61)
 		(descr "Capacitor SMD 0402 (1005 Metric), square (rectangular) end terminal, IPC-7351 nominal with elongated pad for handsoldering. (Body size source: IPC-SM-782 page 76, https://www.pcb-3d.com/wordpress/wp-content/uploads/ipc-sm-782a_amendment_1_and_2.pdf)")
 		(tags "capacitor handsolder")
@@
 	(footprint "Capacitor_SMD:C_0402_1005Metric_Pad0.74x0.62mm_HandSolder"
 		(layer "F.Cu")
-		(at 99.035 84.225)
+		(at 91.2575 76.37)
 		(descr "Capacitor SMD 0402 (1005 Metric), square (rectangular) end terminal, IPC-7351 nominal with elongated pad for handsoldering. (Body size source: IPC-SM-782 page 76, https://www.pcb-3d.com/wordpress/wp-content/uploads/ipc-sm-782a_amendment_1_and_2.pdf)")
 		(tags "capacitor handsolder")
@@
 		(sheetname "/")
 		(sheetfile "10CL006YE144C8G.kicad_sch")
-		(units
-			(unit
-				(name "A")
-				(pins "1" "2")
-			)
-		)
 		(attr smd)
 		(duplicate_pad_numbers_are_jumpers no)
