File: test_boards/10CL006YE144C8G/orig/10CL006YE144C8G.kicad_sch (KiCad schematic)
At the start: 81 parts, among them IC401 10CL006YE144C8G, J401 CL_JTAG, U401 W25Q128JVS, Y401 SG-7050CAN

Commit message: Правки
Parts:
- added C37: 4.7 uF, Capacitor_SMD:C_0603_1608Metric_Pad1.08x0.95mm_HandSolder, symbol Device:C
- C27: renamed from C455; value 4.7 uF -> 100 nF
- renumbered C401 to C1, C410 to C10, C411 to C11, C412 to C12, C432 to C13, C461 to C14, C417 to C15, C418 to C16, C419 to C17, C420 to C18, C421 to C19, C402 to C2, C422 to C20, C423 to C21, C424 to C22, C425 to C23, C426 to C24, C427 to C25, C458 to C26, C429 to C28, C430 to C29, C403 to C3, C414 to C30, C413 to C31, C452 to C32, C416 to C33, C449 to C34, C453 to C35, C456 to C36, C433 to C38, C434 to C39, C404 to C4, C415 to C40, C431 to C41, C428 to C42, C447 to C43, C448 to C44, C450 to C45, C451 to C46, C435 to C47, C436 to C48, C437 to C49, C405 to C5, C438 to C50, C454 to C51, C457 to C52, C459 to C53, C460 to C54, C440 to C55, C442 to C56, C444 to C57, C439 to C58, C446 to C59, C406 to C6, C441 to C60, C443 to C61, C445 to C62, C407 to C7, C408 to C8, C409 to C9, FB401 to FB1, FB402 to FB2, FB403 to FB3, FB404 to FB4, IC401 to IC1, J401 to J1, R404 to R1, R412 to R10, R413 to R11, R414 to R12, R407 to R2, R401 to R3, R402 to R4, R409 to R5, R403 to R6, R408 to R7, R410 to R8, R411 to R9, U401 to U1, Y401 to Y1
Connections:
- net +3V3_VCCIO: now also C37.1
- net GND: now also C37.2
