File: test_boards/Power/Power.kicad_pcb (KiCad board)
At the start: 2 copper layers, 55 parts, among them J201 ±5V In, U201 AMS1117-1.2, U202 AMS1117CD-3.3, U203 LM317_TO-252, U204 LM337_TO252

Commit message: добавлены настройки профилей
Parts:
- moved J201 178.2 mm to (21.1, 62.1), turned to -90 degrees
- moved C201 147.3 mm to (77.4, 50.9), turned to -90 degrees
- moved C203 128.0 mm to (80.9, 48.6), turned to -90 degrees
- moved C211 124.1 mm to (85.5, 48.6), turned to -90 degrees
- moved FB201 118.7 mm to (82.0, 45.1)
- moved C207 108.5 mm to (83.2, 49.3), turned to -90 degrees
Routing:
- net +5V_DIRTY: track 0.00 -> 11.0 mm, vias 0 -> 1
- net GND: track 0.00 -> 9.18 mm, vias 0 -> 4
- net +5V: track 0.00 -> 7.17 mm, vias 0 -> 1
Other:
- copper layers 2 -> 4
