File: test_boards/Power/Power.kicad_pcb (KiCad board)
At the start: 4 copper layers, 55 parts, among them J1 ±5V In, U1 AMS1117-1.2, U2 AMS1117CD-3.3, U3 LM317_TO-252, U4 LM337_TO252

Commit message: Теперь, реестр привязывается к размещению и переименование клона не трогает via и треки
Parts:
- C10, C11, C13, C14, C21, C22: footprint Capacitor_SMD:C_1206_3216Metric_Pad1.33x1.80mm_HandSolder -> Capacitor_SMD:C_0603_1608Metric_Pad1.08x0.95mm_HandSolder
- C23, C24: footprint Capacitor_SMD:C_1206_3216Metric_Pad1.33x1.80mm_HandSolder -> Capacitor_SMD:C_0805_2012Metric_Pad1.18x1.45mm_HandSolder
- moved C2 106.2 mm to (41.2, 58.3), turned to -90 degrees
- moved FB3 91.7 mm to (57.0, 69.1)
- moved C5 89.9 mm to (53.5, 72.6), turned to -90 degrees
- moved FB4 86.7 mm to (58.9, 84.1)
- moved C6 85.6 mm to (55.4, 87.6), turned to -90 degrees
- moved C4 84.7 mm to (44.7, 56.0), turned to -90 degrees
- moved FB2 81.3 mm to (45.8, 52.6)
- moved C12 81.1 mm to (49.2, 56.0), turned to -90 degrees
- moved U1 80.6 mm to (44.3, 70.9)
- moved U2 77.1 mm to (46.1, 86.0)
- moved C15 70.2 mm to (58.5, 71.8), turned to -90 degrees
- moved C16 68.7 mm to (60.4, 86.8), turned to -90 degrees
- moved C8 65.5 mm to (47.0, 56.7), turned to -90 degrees
- moved D6 57.6 mm to (92.5, 53.2), turned to 180 degrees
- moved R4 56.6 mm to (84.8, 53.2), turned to 180 degrees
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Routing:
- net GND: track 9.17 -> 33.5 mm, vias 4 -> 14
- net -5V_DIRTY: track 0.00 -> 11.0 mm, vias 0 -> 1
- net +1V2_DIRTY: track 0.00 -> 7.18 mm, vias 0 -> 1
- net +3V3_DIRTY: track 0.00 -> 7.18 mm, vias 0 -> 1
- net -5V: track 0.00 -> 7.16 mm, vias 0 -> 1
- net +1V2: track 0.00 -> 6.32 mm, vias 0 -> 1
- net +3V3: track 0.00 -> 6.32 mm, vias 0 -> 1

Commit message: Исправил ошибочный manual_position_calculator
Parts:
- removed C1, C2: TAJD107K016RNJ, Capacitor_Tantalum_SMD:CP_EIA-7343-20_Kemet-V_HandSolder
- removed C10, C11, C13, C14, C21, C22: 1 uF, Capacitor_SMD:C_0603_1608Metric_Pad1.08x0.95mm_HandSolder
- removed C12, C15, C16, C17, C18, C19, C20, C25, C26, C3, C4, C9: 100 nF, Capacitor_SMD:C_0603_1608Metric_Pad1.08x0.95mm_HandSolder
- removed C23, C24: 10 uF, Capacitor_SMD:C_0805_2012Metric_Pad1.18x1.45mm_HandSolder
- removed C5, C6: TAJB476K010UNJ, Capacitor_Tantalum_SMD:CP_EIA-3528-12_Kemet-T_HandSolder
- removed C7, C8: 1 uF, Capacitor_SMD:C_1206_3216Metric_Pad1.33x1.80mm_HandSolder
- removed D1, D2, D3, D8, D9: LED, Diode_SMD:D_0805_2012Metric_Pad1.15x1.40mm_HandSolder
- removed D4, D5, D6, D7: D, Diode_SMD:D_SMA_Handsoldering
- removed FB1, FB2: BLM21PG121SN1D, Inductor_SMD:L_0805_2012Metric
- removed FB3, FB4, FB5, FB6: BLM15PD121SN1D, Inductor_SMD:L_0402_1005Metric
- removed J1: ±5V In, Connector_JST:JST_XH_B3B-XH-A_1x03_P2.50mm_Vertical
- removed R1, R2: 470, Resistor_SMD:R_0603_1608Metric_Pad0.98x0.95mm_HandSolder
- removed R3: 330, Resistor_SMD:R_0603_1608Metric_Pad0.98x0.95mm_HandSolder
- removed R4, R5, R6, R7: 240, Resistor_SMD:R_0603_1608Metric_Pad0.98x0.95mm_HandSolder
- removed R8, R9: 220, Resistor_SMD:R_0603_1608Metric_Pad0.98x0.95mm_HandSolder
- removed U1: AMS1117-1.2, Package_TO_SOT_SMD:SOT-223-3_TabPin2
- removed U2: AMS1117CD-3.3, Package_TO_SOT_SMD:TO-252-3_TabPin2
- removed U3: LM317_TO-252, Package_TO_SOT_SMD:TO-252-2
- removed U4: LM337_TO252, Package_TO_SOT_SMD:TO-252-2
Routing:
- net GND: track 33.5 -> 0.00 mm, vias 14 -> 0
- net -5V_DIRTY: track 11.0 -> 0.00 mm, vias 1 -> 0
- net +5V_DIRTY: track 11.0 -> 0.00 mm, vias 1 -> 0
- net +1V2_DIRTY: track 7.18 -> 0.00 mm, vias 1 -> 0
- net +3V3_DIRTY: track 7.18 -> 0.00 mm, vias 1 -> 0
- net +5V: track 7.16 -> 0.00 mm, vias 1 -> 0
- net -5V: track 7.16 -> 0.00 mm, vias 1 -> 0
- net +1V2: track 6.32 -> 0.00 mm, vias 1 -> 0
- net +3V3: track 6.32 -> 0.00 mm, vias 1 -> 0

Commit message: Доработка документации
Parts:
- added C1: TAJD107K016RNJ, Capacitor_Tantalum_SMD:CP_EIA-7343-20_Kemet-V_HandSolder, F.Cu at (151.2, 65.4)
- added C10: 1 uF, Capacitor_SMD:C_0603_1608Metric_Pad1.08x0.95mm_HandSolder, F.Cu at (153.5, 53.1)
- added C11: 1 uF, Capacitor_SMD:C_0603_1608Metric_Pad1.08x0.95mm_HandSolder, F.Cu at (153.5, 55.6)
- added C12: 100 nF, Capacitor_SMD:C_0603_1608Metric_Pad1.08x0.95mm_HandSolder, F.Cu at (153.5, 58.1)
- added C13: 1 uF, Capacitor_SMD:C_0603_1608Metric_Pad1.08x0.95mm_HandSolder, F.Cu at (153.5, 60.6)
- added C14: 1 uF, Capacitor_SMD:C_0603_1608Metric_Pad1.08x0.95mm_HandSolder, F.Cu at (157.9, 45.5)
- added C15: 100 nF, Capacitor_SMD:C_0603_1608Metric_Pad1.08x0.95mm_HandSolder, F.Cu at (157.9, 48.0)
- added C16: 100 nF, Capacitor_SMD:C_0603_1608Metric_Pad1.08x0.95mm_HandSolder, F.Cu at (157.9, 50.6)
- added C17: 100 nF, Capacitor_SMD:C_0603_1608Metric_Pad1.08x0.95mm_HandSolder, F.Cu at (157.9, 53.1)
- added C18: 100 nF, Capacitor_SMD:C_0603_1608Metric_Pad1.08x0.95mm_HandSolder, F.Cu at (157.9, 55.6)
- added C19: 100 nF, Capacitor_SMD:C_0603_1608Metric_Pad1.08x0.95mm_HandSolder, F.Cu at (157.9, 58.1)
- added C2: TAJD107K016RNJ, Capacitor_Tantalum_SMD:CP_EIA-7343-20_Kemet-V_HandSolder, F.Cu at (151.2, 71.3)
- added C20: 100 nF, Capacitor_SMD:C_0603_1608Metric_Pad1.08x0.95mm_HandSolder, F.Cu at (157.9, 60.6)
- added C21: 1 uF, Capacitor_SMD:C_0603_1608Metric_Pad1.08x0.95mm_HandSolder, F.Cu at (162.2, 45.5)
- added C22: 1 uF, Capacitor_SMD:C_0603_1608Metric_Pad1.08x0.95mm_HandSolder, F.Cu at (162.2, 48.0)
- added C23: 10 uF, Capacitor_SMD:C_0805_2012Metric_Pad1.18x1.45mm_HandSolder, F.Cu at (131.5, 78.2)
- added C24: 10 uF, Capacitor_SMD:C_0805_2012Metric_Pad1.18x1.45mm_HandSolder, F.Cu at (131.5, 81.2)
- added C25: 100 nF, Capacitor_SMD:C_0603_1608Metric_Pad1.08x0.95mm_HandSolder, F.Cu at (162.2, 50.6)
- added C26: 100 nF, Capacitor_SMD:C_0603_1608Metric_Pad1.08x0.95mm_HandSolder, F.Cu at (162.2, 53.1)
- added C3: 100 nF, Capacitor_SMD:C_0603_1608Metric_Pad1.08x0.95mm_HandSolder, F.Cu at (153.5, 45.5)
- added C4: 100 nF, Capacitor_SMD:C_0603_1608Metric_Pad1.08x0.95mm_HandSolder, F.Cu at (153.5, 48.0)
- added C5: TAJB476K010UNJ, Capacitor_Tantalum_SMD:CP_EIA-3528-12_Kemet-T_HandSolder, F.Cu at (159.5, 64.7)
- added C6: TAJB476K010UNJ, Capacitor_Tantalum_SMD:CP_EIA-3528-12_Kemet-T_HandSolder, F.Cu at (159.5, 69.0)
- added C7: 1 uF, Capacitor_SMD:C_1206_3216Metric_Pad1.33x1.80mm_HandSolder, F.Cu at (149.1, 75.9)
- added C8: 1 uF, Capacitor_SMD:C_1206_3216Metric_Pad1.33x1.80mm_HandSolder, F.Cu at (149.1, 79.2)
- added C9: 100 nF, Capacitor_SMD:C_0603_1608Metric_Pad1.08x0.95mm_HandSolder, F.Cu at (153.5, 50.6)
- added D1: LED, Diode_SMD:D_0805_2012Metric_Pad1.15x1.40mm_HandSolder, F.Cu at (143.7, 64.0)
- added D2: LED, Diode_SMD:D_0805_2012Metric_Pad1.15x1.40mm_HandSolder, F.Cu at (143.7, 67.0)
- added D3: LED, Diode_SMD:D_0805_2012Metric_Pad1.15x1.40mm_HandSolder, F.Cu at (143.7, 70.1)
- added D4: D, Diode_SMD:D_SMA_Handsoldering, F.Cu at (146.3, 46.6)
- added D5: D, Diode_SMD:D_SMA_Handsoldering, F.Cu at (146.3, 51.1)
- added D6: D, Diode_SMD:D_SMA_Handsoldering, F.Cu at (146.3, 55.7)
- added D7: D, Diode_SMD:D_SMA_Handsoldering, F.Cu at (146.3, 60.2)
- added D8: LED, Diode_SMD:D_0805_2012Metric_Pad1.15x1.40mm_HandSolder, F.Cu at (143.7, 73.1)
- added D9: LED, Diode_SMD:D_0805_2012Metric_Pad1.15x1.40mm_HandSolder, F.Cu at (143.7, 76.2)
- added FB1: BLM21PG121SN1D, Inductor_SMD:L_0805_2012Metric, F.Cu at (136.2, 78.0)
- added FB2: BLM21PG121SN1D, Inductor_SMD:L_0805_2012Metric, F.Cu at (136.2, 80.8)
- added FB3: BLM15PD121SN1D, Inductor_SMD:L_0402_1005Metric, F.Cu at (164.1, 63.5)
- added FB4: BLM15PD121SN1D, Inductor_SMD:L_0402_1005Metric, F.Cu at (164.1, 65.5)
- added FB5: BLM15PD121SN1D, Inductor_SMD:L_0402_1005Metric, F.Cu at (164.1, 67.5)
- added FB6: BLM15PD121SN1D, Inductor_SMD:L_0402_1005Metric, F.Cu at (164.1, 69.4)
- added J1: ±5V In, Connector_JST:JST_XH_B3B-XH-A_1x03_P2.50mm_Vertical, F.Cu at (37.3, 46.2)
- added R1: 470, Resistor_SMD:R_0603_1608Metric_Pad0.98x0.95mm_HandSolder, F.Cu at (162.2, 55.6)
- added R2: 470, Resistor_SMD:R_0603_1608Metric_Pad0.98x0.95mm_HandSolder, F.Cu at (162.2, 58.1)
- added R3: 330, Resistor_SMD:R_0603_1608Metric_Pad0.98x0.95mm_HandSolder, F.Cu at (162.2, 60.6)
- added R4: 240, Resistor_SMD:R_0603_1608Metric_Pad0.98x0.95mm_HandSolder, F.Cu at (166.6, 45.5)
- added R5: 240, Resistor_SMD:R_0603_1608Metric_Pad0.98x0.95mm_HandSolder, F.Cu at (166.6, 48.0)
- added R6: 240, Resistor_SMD:R_0603_1608Metric_Pad0.98x0.95mm_HandSolder, F.Cu at (166.6, 50.6)
- added R7: 240, Resistor_SMD:R_0603_1608Metric_Pad0.98x0.95mm_HandSolder, F.Cu at (166.6, 53.1)
- added R8: 220, Resistor_SMD:R_0603_1608Metric_Pad0.98x0.95mm_HandSolder, F.Cu at (166.6, 55.6)
- added R9: 220, Resistor_SMD:R_0603_1608Metric_Pad0.98x0.95mm_HandSolder, F.Cu at (166.6, 58.1)
- added U1: AMS1117-1.2, Package_TO_SOT_SMD:SOT-223-3_TabPin2, F.Cu at (161.2, 75.4)
- added U2: AMS1117CD-3.3, Package_TO_SOT_SMD:TO-252-3_TabPin2, F.Cu at (136.0, 48.5)
- added U3: LM317_TO-252, Package_TO_SOT_SMD:TO-252-2, F.Cu at (136.0, 56.6)
- added U4: LM337_TO252, Package_TO_SOT_SMD:TO-252-2, F.Cu at (136.0, 64.8)
