File: test_boards/3CH-AWG-TIA/power.kicad_sch (KiCad schematic)
At the start: 55 parts, among them J1 ±5V In, U1 AMS1117-1.2, U2 AMS1117CD-3.3, U3 LM317_TO-252, U4 LM337_TO252

Commit message: Добавлен anchor_role в генерируемые шаблоны
Parts:
- added D3: LED, Diode_SMD:D_0805_2012Metric_Pad1.15x1.40mm_HandSolder, symbol Device:LED
- added R3: 50, Resistor_SMD:R_0603_1608Metric_Pad0.98x0.95mm_HandSolder, symbol Device:R
- C1, C3, C7, C9, FB1: Cluster (none) -> In_Pi_Filter_Pos
- C10, C13, C15, C5: Cluster (none) -> Pi_Filter_Out_1V2
- C11, C14, C16, C6, FB4: Cluster (none) -> Pi_Filter_Out_3V3
- C12, C2, C4, C8, FB2: Cluster (none) -> In_Pi_Filter_Neg
- C17, C23: Cluster (none) -> LDO_Subsystem_P2V5
- C18, C21, C25, FB5: Cluster (none) -> Out_Pi_Filter_P2V5
- C19, C22, C26, FB6: Cluster (none) -> Out_Pi_Filter_N2V5
- C20, C24: Cluster (none) -> LDO_Subsystem_N2V5
- D1, R1: Cluster (none) -> Led_P5V
- D10: renamed from D9; Cluster (none) -> Led_P2V5
- D2, R2: Cluster (none) -> Led_N5V
- D4: renamed from D3; Cluster (none) -> Led_3V3
- D5: renamed from D4; Cluster (none) -> LDO_Subsystem_P2V5
- D6: renamed from D5; Cluster (none) -> LDO_Subsystem_N2V5
- D7: renamed from D6; Cluster (none) -> LDO_Subsystem_P2V5
- D8: renamed from D7; Cluster (none) -> LDO_Subsystem_N2V5
- D9: renamed from D8; Cluster (none) -> Led_N2V5
- R10: renamed from R9; Cluster (none) -> Led_P2V5
- R4: renamed from R3; Cluster (none) -> Led_3V3
- R5: renamed from R4; Cluster (none) -> LDO_Subsystem_P2V5
- R6: renamed from R5; Cluster (none) -> LDO_Subsystem_N2V5
- R7: renamed from R6; Cluster (none) -> LDO_Subsystem_P2V5
- R8: renamed from R7; Cluster (none) -> LDO_Subsystem_N2V5
- R9: renamed from R8; Cluster (none) -> Led_N2V5
- U1: Role LDO -> LDO_1V2
- U2: Role LDO -> LDO_3V3
- U3: Role LDO_ADJ -> LDO_ADJ_P2V5
- U4: Role LDO_ADJ -> LDO_ADJ_N2V5
Connections:
- net +1V2: now also R3.2
- net GND: now also D3.1 (K)
- new net +1V2_LED: D3.2 (A), R3.1
