File: test_boards/3CH-AWG-TIA/power_pm18v.kicad_sch (KiCad schematic)
At the start: 5 parts, among them J2 +-18V_PA

Commit message: Добавлен anchor_role в генерируемые шаблоны
Parts:
- C27, C29: Cluster (none) -> In_Filter_P18V
- C28, C30: Cluster (none) -> In_Filter_N18V
Changed lines of the file:
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@@
 		(dnp no)
 		(fields_autoplaced yes)
-		(property "Reference" "#PWR049"
+		(property "Reference" "#PWR051"
 			(at 93.98 107.95 0)
 			(hide yes)
@@
 			(project "3CH-AWG-TIA"
 				(path "/1e22769e-c24b-4bb1-9c9f-ec579d192217/1e5ef2d5-403e-4249-9e10-59c2a2eeeae0"
-					(reference "#PWR049")
+					(reference "#PWR051")
 					(unit 1)
 				)
@@
 			)
 		)
+		(property "Cluster" "In_Filter_N18V"
+			(at 93.98 97.79 0)
+			(hide yes)
+			(show_name no)
+			(do_not_autoplace no)
+			(effects
+				(font
+					(size 1.27 1.27)
+				)
+			)
+		)
 		(pin "1"
 		)
@@
 			)
 		)
+		(property "Cluster" "In_Filter_P18V"
+			(at 93.98 76.2 0)
+			(hide yes)
+			(show_name no)
+			(do_not_autoplace no)
+			(effects
+				(font
+					(size 1.27 1.27)
+				)
+			)
+		)
 		(pin "1"
 		)
@@
 		(dnp no)
 		(fields_autoplaced yes)
-		(property "Reference" "#PWR047"
+		(property "Reference" "#PWR049"
 			(at 74.93 97.79 0)
 			(hide yes)
@@
 			(project "3CH-AWG-TIA"
 				(path "/1e22769e-c24b-4bb1-9c9f-ec579d192217/1e5ef2d5-403e-4249-9e10-59c2a2eeeae0"
-					(reference "#PWR047")
+					(reference "#PWR049")
 					(unit 1)
 				)
@@
 			)
 		)
+		(property "Cluster" "In_Filter_P18V"
+			(at 78.74 76.2 0)
+			(hide yes)
+			(show_name no)
+			(do_not_autoplace no)
+			(effects
+				(font
+					(size 1.27 1.27)
+				)
+			)
+		)
 		(pin "2"
 		)
@@
 		(dnp no)
 		(fields_autoplaced yes)
-		(property "Reference" "#PWR048"
+		(property "Reference" "#PWR050"
 			(at 93.98 86.36 0)
 			(hide yes)
@@
 			(project "3CH-AWG-TIA"
 				(path "/1e22769e-c24b-4bb1-9c9f-ec579d192217/1e5ef2d5-403e-4249-9e10-59c2a2eeeae0"
-					(reference "#PWR048")
+					(reference "#PWR050")
 					(unit 1)
 				)
@@
 		(dnp no)
 		(fields_autoplaced yes)
-		(property "Reference" "#PWR046"
+		(property "Reference" "#PWR048"
 			(at 74.93 76.2 0)
 			(hide yes)
@@
 			(project "3CH-AWG-TIA"
 				(path "/1e22769e-c24b-4bb1-9c9f-ec579d192217/1e5ef2d5-403e-4249-9e10-59c2a2eeeae0"
-					(reference "#PWR046")
+					(reference "#PWR048")
 					(unit 1)
 				)
@@
 			(at 78.74 97.79 0)
 			(hide yes)
+			(show_name no)
+			(do_not_autoplace no)
+			(effects
+				(font
+					(size 1.27 1.27)
+				)
+			)
+		)
+		(property "Cluster" "In_Filter_N18V"
+			(at 78.74 97.79 0)
+			(hide yes)
