File: test_boards/3CH-AWG-TIA/dac.kicad_sch (KiCad schematic)
At the start: 20 parts, among them IC2 AD9707BCPZ

Commit message: Добавлен anchor_role в генерируемые шаблоны
Parts:
- renumbered R32 to R33, R33 to R34, R34 to R35

Commit message: Теперь можно использовать  anchor_role, anchor_cluster в thermal_via_array и manual positions
Parts:
- renumbered C96 to C105, C97 to C106, C98 to C107, C99 to C108, C100 to C109, C101 to C110, C102 to C111, C103 to C112, C104 to C113, C105 to C114, C106 to C115, C107 to C116, C108 to C117
