File: test_boards/3CH-AWG-TIA/op_amp.kicad_sch (KiCad schematic)
At the start: 15 parts, among them U6 ADA4807-2ARM

Commit message: Добавлен anchor_role в генерируемые шаблоны
Parts:
- renumbered R35 to R36, R36 to R37, R37 to R38, R38 to R39
Changed lines of the file:
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@@
 		(in_pos_files yes)
 		(dnp no)
-		(property "Reference" "R37"
+		(property "Reference" "R38"
 			(at 180.34 78.74 90)
 			(show_name no)
@@
 			(project "3CH-AWG-TIA"
 				(path "/1e22769e-c24b-4bb1-9c9f-ec579d192217/37fadcfc-2053-465b-a57f-61f3ae87f57a/946f3b70-3e91-410c-9ab8-56896ff295fa"
-					(reference "R53")
-					(unit 1)
-				)
-				(path "/1e22769e-c24b-4bb1-9c9f-ec579d192217/6b018f07-dde5-4cc8-ba46-360bc68cf3d3/946f3b70-3e91-410c-9ab8-56896ff295fa"
-					(reference "R69")
-					(unit 1)
-				)
-				(path "/1e22769e-c24b-4bb1-9c9f-ec579d192217/fb16a0a4-f706-49de-9d7e-e9bca2583031/946f3b70-3e91-410c-9ab8-56896ff295fa"
-					(reference "R37")
+					(reference "R54")
+					(unit 1)
+				)
+				(path "/1e22769e-c24b-4bb1-9c9f-ec579d192217/6b018f07-dde5-4cc8-ba46-360bc68cf3d3/946f3b70-3e91-410c-9ab8-56896ff295fa"
+					(reference "R70")
+					(unit 1)
+				)
+				(path "/1e22769e-c24b-4bb1-9c9f-ec579d192217/fb16a0a4-f706-49de-9d7e-e9bca2583031/946f3b70-3e91-410c-9ab8-56896ff295fa"
+					(reference "R38")
 					(unit 1)
 				)
@@
 		(dnp no)
 		(fields_autoplaced yes)
-		(property "Reference" "#PWR0102"
+		(property "Reference" "#PWR0104"
 			(at 33.02 71.12 0)
 			(hide yes)
@@
 			(project "3CH-AWG-TIA"
 				(path "/1e22769e-c24b-4bb1-9c9f-ec579d192217/37fadcfc-2053-465b-a57f-61f3ae87f57a/946f3b70-3e91-410c-9ab8-56896ff295fa"
-					(reference "#PWR0132")
-					(unit 1)
-				)
-				(path "/1e22769e-c24b-4bb1-9c9f-ec579d192217/6b018f07-dde5-4cc8-ba46-360bc68cf3d3/946f3b70-3e91-410c-9ab8-56896ff295fa"
-					(reference "#PWR0162")
-					(unit 1)
-				)
-				(path "/1e22769e-c24b-4bb1-9c9f-ec579d192217/fb16a0a4-f706-49de-9d7e-e9bca2583031/946f3b70-3e91-410c-9ab8-56896ff295fa"
-					(reference "#PWR0102")
+					(reference "#PWR0134")
+					(unit 1)
+				)
+				(path "/1e22769e-c24b-4bb1-9c9f-ec579d192217/6b018f07-dde5-4cc8-ba46-360bc68cf3d3/946f3b70-3e91-410c-9ab8-56896ff295fa"
+					(reference "#PWR0164")
+					(unit 1)
+				)
+				(path "/1e22769e-c24b-4bb1-9c9f-ec579d192217/fb16a0a4-f706-49de-9d7e-e9bca2583031/946f3b70-3e91-410c-9ab8-56896ff295fa"
+					(reference "#PWR0104")
 					(unit 1)
 				)
@@
 		(dnp no)
 		(fields_autoplaced yes)
-		(property "Reference" "#PWR0103"
+		(property "Reference" "#PWR0105"
 			(at 101.6 53.34 0)
 			(hide yes)
@@
 			(project "3CH-AWG-TIA"
 				(path "/1e22769e-c24b-4bb1-9c9f-ec579d192217/37fadcfc-2053-465b-a57f-61f3ae87f57a/946f3b70-3e91-410c-9ab8-56896ff295fa"
-					(reference "#PWR0133")
-					(unit 1)
-				)
-				(path "/1e22769e-c24b-4bb1-9c9f-ec579d192217/6b018f07-dde5-4cc8-ba46-360bc68cf3d3/946f3b70-3e91-410c-9ab8-56896ff295fa"
-					(reference "#PWR0163")
-					(unit 1)
-				)
-				(path "/1e22769e-c24b-4bb1-9c9f-ec579d192217/fb16a0a4-f706-49de-9d7e-e9bca2583031/946f3b70-3e91-410c-9ab8-56896ff295fa"
-					(reference "#PWR0103")
+					(reference "#PWR0135")
+					(unit 1)
+				)
+				(path "/1e22769e-c24b-4bb1-9c9f-ec579d192217/6b018f07-dde5-4cc8-ba46-360bc68cf3d3/946f3b70-3e91-410c-9ab8-56896ff295fa"
+					(reference "#PWR0165")
+					(unit 1)
+				)
+				(path "/1e22769e-c24b-4bb1-9c9f-ec579d192217/fb16a0a4-f706-49de-9d7e-e9bca2583031/946f3b70-3e91-410c-9ab8-56896ff295fa"
+					(reference "#PWR0105")
 					(unit 1)
 				)
@@
 		(in_pos_files yes)
 		(dnp no)
-		(property "Reference" "R36"
+		(property "Reference" "R37"
 			(at 143.51 63.5 90)
 			(show_name no)
@@
 			(project "3CH-AWG-TIA"
 				(path "/1e22769e-c24b-4bb1-9c9f-ec579d192217/37fadcfc-2053-465b-a57f-61f3ae87f57a/946f3b70-3e91-410c-9ab8-56896ff295fa"
-					(reference "R52")
-					(unit 1)
-				)
-				(path "/1e22769e-c24b-4bb1-9c9f-ec579d192217/6b018f07-dde5-4cc8-ba46-360bc68cf3d3/946f3b70-3e91-410c-9ab8-56896ff295fa"
-					(reference "R68")
-					(unit 1)
-				)
-				(path "/1e22769e-c24b-4bb1-9c9f-ec579d192217/fb16a0a4-f706-49de-9d7e-e9bca2583031/946f3b70-3e91-410c-9ab8-56896ff295fa"
-					(reference "R36")
+					(reference "R53")
+					(unit 1)
+				)
+				(path "/1e22769e-c24b-4bb1-9c9f-ec579d192217/6b018f07-dde5-4cc8-ba46-360bc68cf3d3/946f3b70-3e91-410c-9ab8-56896ff295fa"
+					(reference "R69")
+					(unit 1)
+				)
+				(path "/1e22769e-c24b-4bb1-9c9f-ec579d192217/fb16a0a4-f706-49de-9d7e-e9bca2583031/946f3b70-3e91-410c-9ab8-56896ff295fa"
+					(reference "R37")
 					(unit 1)
 				)
@@
 		(dnp no)
 		(fields_autoplaced yes)
-		(property "Reference" "#PWR0104"
+		(property "Reference" "#PWR0106"
 			(at 101.6 81.28 0)
 			(hide yes)
@@
 			(project "3CH-AWG-TIA"
 				(path "/1e22769e-c24b-4bb1-9c9f-ec579d192217/37fadcfc-2053-465b-a57f-61f3ae87f57a/946f3b70-3e91-410c-9ab8-56896ff295fa"
-					(reference "#PWR0134")
-					(unit 1)
-				)
-				(path "/1e22769e-c24b-4bb1-9c9f-ec579d192217/6b018f07-dde5-4cc8-ba46-360bc68cf3d3/946f3b70-3e91-410c-9ab8-56896ff295fa"
-					(reference "#PWR0164")
-					(unit 1)
-				)
-				(path "/1e22769e-c24b-4bb1-9c9f-ec579d192217/fb16a0a4-f706-49de-9d7e-e9bca2583031/946f3b70-3e91-410c-9ab8-56896ff295fa"
-					(reference "#PWR0104")
+					(reference "#PWR0136")
+					(unit 1)
+				)
+				(path "/1e22769e-c24b-4bb1-9c9f-ec579d192217/6b018f07-dde5-4cc8-ba46-360bc68cf3d3/946f3b70-3e91-410c-9ab8-56896ff295fa"
+					(reference "#PWR0166")
+					(unit 1)
+				)
+				(path "/1e22769e-c24b-4bb1-9c9f-ec579d192217/fb16a0a4-f706-49de-9d7e-e9bca2583031/946f3b70-3e91-410c-9ab8-56896ff295fa"
+					(reference "#PWR0106")
 					(unit 1)
 				)
@@
 		(in_pos_files yes)
 		(dnp no)
-		(property "Reference" "R35"
+		(property "Reference" "R36"
 			(at 143.51 31.75 90)
 			(show_name no)
@@
 			(project "3CH-AWG-TIA"
 				(path "/1e22769e-c24b-4bb1-9c9f-ec579d192217/37fadcfc-2053-465b-a57f-61f3ae87f57a/946f3b70-3e91-410c-9ab8-56896ff295fa"
-					(reference "R51")
-					(unit 1)
-				)
-				(path "/1e22769e-c24b-4bb1-9c9f-ec579d192217/6b018f07-dde5-4cc8-ba46-360bc68cf3d3/946f3b70-3e91-410c-9ab8-56896ff295fa"
-					(reference "R67")
-					(unit 1)
-				)
-				(path "/1e22769e-c24b-4bb1-9c9f-ec579d192217/fb16a0a4-f706-49de-9d7e-e9bca2583031/946f3b70-3e91-410c-9ab8-56896ff295fa"
-					(reference "R35")
+					(reference "R52")
+					(unit 1)
+				)
+				(path "/1e22769e-c24b-4bb1-9c9f-ec579d192217/6b018f07-dde5-4cc8-ba46-360bc68cf3d3/946f3b70-3e91-410c-9ab8-56896ff295fa"
+					(reference "R68")
+					(unit 1)
+				)
+				(path "/1e22769e-c24b-4bb1-9c9f-ec579d192217/fb16a0a4-f706-49de-9d7e-e9bca2583031/946f3b70-3e91-410c-9ab8-56896ff295fa"
+					(reference "R36")
 					(unit 1)
 				)
@@
 		(dnp no)
 		(fields_autoplaced yes)
-		(property "Reference" "#PWR0101"
+		(property "Reference" "#PWR0103"
 			(at 33.02 43.18 0)
 			(hide yes)
@@
 			(project "3CH-AWG-TIA"
 				(path "/1e22769e-c24b-4bb1-9c9f-ec579d192217/37fadcfc-2053-465b-a57f-61f3ae87f57a/946f3b70-3e91-410c-9ab8-56896ff295fa"
-					(reference "#PWR0131")
-					(unit 1)
-				)
-				(path "/1e22769e-c24b-4bb1-9c9f-ec579d192217/6b018f07-dde5-4cc8-ba46-360bc68cf3d3/946f3b70-3e91-410c-9ab8-56896ff295fa"
-					(reference "#PWR0161")
-					(unit 1)
-				)
-				(path "/1e22769e-c24b-4bb1-9c9f-ec579d192217/fb16a0a4-f706-49de-9d7e-e9bca2583031/946f3b70-3e91-410c-9ab8-56896ff295fa"
-					(reference "#PWR0101")
+					(reference "#PWR0133")
+					(unit 1)
+				)
+				(path "/1e22769e-c24b-4bb1-9c9f-ec579d192217/6b018f07-dde5-4cc8-ba46-360bc68cf3d3/946f3b70-3e91-410c-9ab8-56896ff295fa"
+					(reference "#PWR0163")
+					(unit 1)
+				)
+				(path "/1e22769e-c24b-4bb1-9c9f-ec579d192217/fb16a0a4-f706-49de-9d7e-e9bca2583031/946f3b70-3e91-410c-9ab8-56896ff295fa"
+					(reference "#PWR0103")
 					(unit 1)
 				)
@@
 		(in_pos_files yes)
 		(dnp no)
-		(property "Reference" "R38"
+		(property "Reference" "R39"
 			(at 181.61 48.26 90)
 			(show_name no)
@@
 			(project "3CH-AWG-TIA"
 				(path "/1e22769e-c24b-4bb1-9c9f-ec579d192217/37fadcfc-2053-465b-a57f-61f3ae87f57a/946f3b70-3e91-410c-9ab8-56896ff295fa"
-					(reference "R54")
-					(unit 1)
-				)
-				(path "/1e22769e-c24b-4bb1-9c9f-ec579d192217/6b018f07-dde5-4cc8-ba46-360bc68cf3d3/946f3b70-3e91-410c-9ab8-56896ff295fa"
-					(reference "R70")
-					(unit 1)
-				)
-				(path "/1e22769e-c24b-4bb1-9c9f-ec579d192217/fb16a0a4-f706-49de-9d7e-e9bca2583031/946f3b70-3e91-410c-9ab8-56896ff295fa"
-					(reference "R38")
-					(unit 1)
-				)
+					(reference "R55")
+					(unit 1)
+				)
+				(path "/1e22769e-c24b-4bb1-9c9f-ec579d192217/6b018f07-dde5-4cc8-ba46-360bc68cf3d3/946f3b70-3e91-410c-9ab8-56896ff295fa"
+					(reference "R71")
+					(unit 1)
+				)
+				(path "/1e22769e-c24b-4bb1-9c9f-ec579d192217/fb16a0a4-f706-49de-9d7e-e9bca2583031/946f3b70-3e91-410c-9ab8-56896ff295fa"
+					(reference "R39")
+					(unit 1)
+				)

Commit message: Теперь можно использовать  anchor_role, anchor_cluster в thermal_via_array и manual positions
Parts:
- renumbered C109 to C118, C110 to C119, C111 to C120, C112 to C121, C113 to C122, C114 to C123, C115 to C124, C116 to C125
Changed lines of the file:
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@@
 		(dnp no)
 		(fields_autoplaced yes)
-		(property "Reference" "C114"
+		(property "Reference" "C123"
 			(at 91.44 69.8499 0)
 			(show_name no)
@@
 			(project "3CH-AWG-TIA"
 				(path "/1e22769e-c24b-4bb1-9c9f-ec579d192217/37fadcfc-2053-465b-a57f-61f3ae87f57a/946f3b70-3e91-410c-9ab8-56896ff295fa"
-					(reference "C148")
-					(unit 1)
-				)
-				(path "/1e22769e-c24b-4bb1-9c9f-ec579d192217/6b018f07-dde5-4cc8-ba46-360bc68cf3d3/946f3b70-3e91-410c-9ab8-56896ff295fa"
-					(reference "C182")
-					(unit 1)
-				)
-				(path "/1e22769e-c24b-4bb1-9c9f-ec579d192217/fb16a0a4-f706-49de-9d7e-e9bca2583031/946f3b70-3e91-410c-9ab8-56896ff295fa"
-					(reference "C114")
+					(reference "C157")
+					(unit 1)
+				)
+				(path "/1e22769e-c24b-4bb1-9c9f-ec579d192217/6b018f07-dde5-4cc8-ba46-360bc68cf3d3/946f3b70-3e91-410c-9ab8-56896ff295fa"
+					(reference "C191")
+					(unit 1)
+				)
+				(path "/1e22769e-c24b-4bb1-9c9f-ec579d192217/fb16a0a4-f706-49de-9d7e-e9bca2583031/946f3b70-3e91-410c-9ab8-56896ff295fa"
+					(reference "C123")
 					(unit 1)
 				)
@@
 		(dnp no)
 		(fields_autoplaced yes)
-		(property "Reference" "C116"
+		(property "Reference" "C125"
 			(at 105.41 69.8499 0)
 			(show_name no)
@@
 			(project "3CH-AWG-TIA"
 				(path "/1e22769e-c24b-4bb1-9c9f-ec579d192217/37fadcfc-2053-465b-a57f-61f3ae87f57a/946f3b70-3e91-410c-9ab8-56896ff295fa"
-					(reference "C150")
-					(unit 1)
-				)
-				(path "/1e22769e-c24b-4bb1-9c9f-ec579d192217/6b018f07-dde5-4cc8-ba46-360bc68cf3d3/946f3b70-3e91-410c-9ab8-56896ff295fa"
-					(reference "C184")
-					(unit 1)
-				)
-				(path "/1e22769e-c24b-4bb1-9c9f-ec579d192217/fb16a0a4-f706-49de-9d7e-e9bca2583031/946f3b70-3e91-410c-9ab8-56896ff295fa"
-					(reference "C116")
+					(reference "C159")
+					(unit 1)
+				)
+				(path "/1e22769e-c24b-4bb1-9c9f-ec579d192217/6b018f07-dde5-4cc8-ba46-360bc68cf3d3/946f3b70-3e91-410c-9ab8-56896ff295fa"
+					(reference "C193")
+					(unit 1)
+				)
+				(path "/1e22769e-c24b-4bb1-9c9f-ec579d192217/fb16a0a4-f706-49de-9d7e-e9bca2583031/946f3b70-3e91-410c-9ab8-56896ff295fa"
+					(reference "C125")
 					(unit 1)
 				)
@@
 		(dnp no)
 		(fields_autoplaced yes)
-		(property "Reference" "C112"
+		(property "Reference" "C121"
 			(at 50.8 69.8499 0)
 			(show_name no)
@@
 			(project "3CH-AWG-TIA"
 				(path "/1e22769e-c24b-4bb1-9c9f-ec579d192217/37fadcfc-2053-465b-a57f-61f3ae87f57a/946f3b70-3e91-410c-9ab8-56896ff295fa"
-					(reference "C146")
-					(unit 1)
-				)
-				(path "/1e22769e-c24b-4bb1-9c9f-ec579d192217/6b018f07-dde5-4cc8-ba46-360bc68cf3d3/946f3b70-3e91-410c-9ab8-56896ff295fa"
-					(reference "C180")
-					(unit 1)
-				)
-				(path "/1e22769e-c24b-4bb1-9c9f-ec579d192217/fb16a0a4-f706-49de-9d7e-e9bca2583031/946f3b70-3e91-410c-9ab8-56896ff295fa"
-					(reference "C112")
+					(reference "C155")
+					(unit 1)
+				)
+				(path "/1e22769e-c24b-4bb1-9c9f-ec579d192217/6b018f07-dde5-4cc8-ba46-360bc68cf3d3/946f3b70-3e91-410c-9ab8-56896ff295fa"
+					(reference "C189")
+					(unit 1)
+				)
+				(path "/1e22769e-c24b-4bb1-9c9f-ec579d192217/fb16a0a4-f706-49de-9d7e-e9bca2583031/946f3b70-3e91-410c-9ab8-56896ff295fa"
+					(reference "C121")
 					(unit 1)
 				)
@@
 		(dnp no)
 		(fields_autoplaced yes)
-		(property "Reference" "C113"
+		(property "Reference" "C122"
 			(at 91.44 41.9099 0)
 			(show_name no)
@@
 			(project "3CH-AWG-TIA"
 				(path "/1e22769e-c24b-4bb1-9c9f-ec579d192217/37fadcfc-2053-465b-a57f-61f3ae87f57a/946f3b70-3e91-410c-9ab8-56896ff295fa"
-					(reference "C147")
-					(unit 1)
-				)
-				(path "/1e22769e-c24b-4bb1-9c9f-ec579d192217/6b018f07-dde5-4cc8-ba46-360bc68cf3d3/946f3b70-3e91-410c-9ab8-56896ff295fa"
-					(reference "C181")
-					(unit 1)
-				)
-				(path "/1e22769e-c24b-4bb1-9c9f-ec579d192217/fb16a0a4-f706-49de-9d7e-e9bca2583031/946f3b70-3e91-410c-9ab8-56896ff295fa"
-					(reference "C113")
+					(reference "C156")
+					(unit 1)
+				)
+				(path "/1e22769e-c24b-4bb1-9c9f-ec579d192217/6b018f07-dde5-4cc8-ba46-360bc68cf3d3/946f3b70-3e91-410c-9ab8-56896ff295fa"
+					(reference "C190")
+					(unit 1)
+				)
+				(path "/1e22769e-c24b-4bb1-9c9f-ec579d192217/fb16a0a4-f706-49de-9d7e-e9bca2583031/946f3b70-3e91-410c-9ab8-56896ff295fa"
+					(reference "C122")
 					(unit 1)
 				)
@@
 		(dnp no)
 		(fields_autoplaced yes)
-		(property "Reference" "C115"
+		(property "Reference" "C124"
 			(at 105.41 41.9099 0)
 			(show_name no)
@@
 			(project "3CH-AWG-TIA"
 				(path "/1e22769e-c24b-4bb1-9c9f-ec579d192217/37fadcfc-2053-465b-a57f-61f3ae87f57a/946f3b70-3e91-410c-9ab8-56896ff295fa"
-					(reference "C149")
-					(unit 1)
-				)
-				(path "/1e22769e-c24b-4bb1-9c9f-ec579d192217/6b018f07-dde5-4cc8-ba46-360bc68cf3d3/946f3b70-3e91-410c-9ab8-56896ff295fa"
-					(reference "C183")
-					(unit 1)
-				)
-				(path "/1e22769e-c24b-4bb1-9c9f-ec579d192217/fb16a0a4-f706-49de-9d7e-e9bca2583031/946f3b70-3e91-410c-9ab8-56896ff295fa"
-					(reference "C115")
+					(reference "C158")
+					(unit 1)
+				)
+				(path "/1e22769e-c24b-4bb1-9c9f-ec579d192217/6b018f07-dde5-4cc8-ba46-360bc68cf3d3/946f3b70-3e91-410c-9ab8-56896ff295fa"
+					(reference "C192")
+					(unit 1)
+				)
+				(path "/1e22769e-c24b-4bb1-9c9f-ec579d192217/fb16a0a4-f706-49de-9d7e-e9bca2583031/946f3b70-3e91-410c-9ab8-56896ff295fa"
+					(reference "C124")
 					(unit 1)
 				)
@@
 		(dnp no)
 		(fields_autoplaced yes)
-		(property "Reference" "C109"
+		(property "Reference" "C118"
 			(at 36.83 41.9099 0)
 			(show_name no)
@@
 			(project "3CH-AWG-TIA"
 				(path "/1e22769e-c24b-4bb1-9c9f-ec579d192217/37fadcfc-2053-465b-a57f-61f3ae87f57a/946f3b70-3e91-410c-9ab8-56896ff295fa"
-					(reference "C143")
-					(unit 1)
-				)
-				(path "/1e22769e-c24b-4bb1-9c9f-ec579d192217/6b018f07-dde5-4cc8-ba46-360bc68cf3d3/946f3b70-3e91-410c-9ab8-56896ff295fa"
-					(reference "C177")
-					(unit 1)
-				)
-				(path "/1e22769e-c24b-4bb1-9c9f-ec579d192217/fb16a0a4-f706-49de-9d7e-e9bca2583031/946f3b70-3e91-410c-9ab8-56896ff295fa"
-					(reference "C109")
+					(reference "C152")
+					(unit 1)
+				)
+				(path "/1e22769e-c24b-4bb1-9c9f-ec579d192217/6b018f07-dde5-4cc8-ba46-360bc68cf3d3/946f3b70-3e91-410c-9ab8-56896ff295fa"
+					(reference "C186")
+					(unit 1)
+				)
+				(path "/1e22769e-c24b-4bb1-9c9f-ec579d192217/fb16a0a4-f706-49de-9d7e-e9bca2583031/946f3b70-3e91-410c-9ab8-56896ff295fa"
+					(reference "C118")
 					(unit 1)
 				)
@@
 		(dnp no)
 		(fields_autoplaced yes)
-		(property "Reference" "C110"
+		(property "Reference" "C119"
 			(at 36.83 69.8499 0)
 			(show_name no)
@@
 			(project "3CH-AWG-TIA"
 				(path "/1e22769e-c24b-4bb1-9c9f-ec579d192217/37fadcfc-2053-465b-a57f-61f3ae87f57a/946f3b70-3e91-410c-9ab8-56896ff295fa"
-					(reference "C144")
-					(unit 1)
-				)
-				(path "/1e22769e-c24b-4bb1-9c9f-ec579d192217/6b018f07-dde5-4cc8-ba46-360bc68cf3d3/946f3b70-3e91-410c-9ab8-56896ff295fa"
-					(reference "C178")
-					(unit 1)
-				)
-				(path "/1e22769e-c24b-4bb1-9c9f-ec579d192217/fb16a0a4-f706-49de-9d7e-e9bca2583031/946f3b70-3e91-410c-9ab8-56896ff295fa"
-					(reference "C110")
+					(reference "C153")
+					(unit 1)
+				)
+				(path "/1e22769e-c24b-4bb1-9c9f-ec579d192217/6b018f07-dde5-4cc8-ba46-360bc68cf3d3/946f3b70-3e91-410c-9ab8-56896ff295fa"
+					(reference "C187")
+					(unit 1)
+				)
+				(path "/1e22769e-c24b-4bb1-9c9f-ec579d192217/fb16a0a4-f706-49de-9d7e-e9bca2583031/946f3b70-3e91-410c-9ab8-56896ff295fa"
+					(reference "C119")
 					(unit 1)
 				)
@@
 		(dnp no)
 		(fields_autoplaced yes)
-		(property "Reference" "C111"
+		(property "Reference" "C120"
 			(at 50.8 41.9099 0)
 			(show_name no)
@@
 			(project "3CH-AWG-TIA"
 				(path "/1e22769e-c24b-4bb1-9c9f-ec579d192217/37fadcfc-2053-465b-a57f-61f3ae87f57a/946f3b70-3e91-410c-9ab8-56896ff295fa"
-					(reference "C145")
-					(unit 1)
-				)
-				(path "/1e22769e-c24b-4bb1-9c9f-ec579d192217/6b018f07-dde5-4cc8-ba46-360bc68cf3d3/946f3b70-3e91-410c-9ab8-56896ff295fa"
-					(reference "C179")
-					(unit 1)
-				)
-				(path "/1e22769e-c24b-4bb1-9c9f-ec579d192217/fb16a0a4-f706-49de-9d7e-e9bca2583031/946f3b70-3e91-410c-9ab8-56896ff295fa"
-					(reference "C111")
-					(unit 1)
-				)
+					(reference "C154")
+					(unit 1)
+				)
+				(path "/1e22769e-c24b-4bb1-9c9f-ec579d192217/6b018f07-dde5-4cc8-ba46-360bc68cf3d3/946f3b70-3e91-410c-9ab8-56896ff295fa"
+					(reference "C188")
+					(unit 1)
+				)
+				(path "/1e22769e-c24b-4bb1-9c9f-ec579d192217/fb16a0a4-f706-49de-9d7e-e9bca2583031/946f3b70-3e91-410c-9ab8-56896ff295fa"
+					(reference "C120")
+					(unit 1)
+				)
