File: test_boards/3CH-AWG-TIA/power_amp.kicad_sch (KiCad schematic)
At the start: 24 parts, among them J4 Signal Out, U7 PC817, U8 ADA4870ARRZ

Commit message: Добавлен anchor_role в генерируемые шаблоны
Parts:
- renumbered D10 to D11, D11 to D12, R39 to R40, R40 to R41, R41 to R42, R42 to R43, R43 to R44, R44 to R45

Commit message: Теперь можно использовать  anchor_role, anchor_cluster в thermal_via_array и manual positions
Parts:
- renumbered C117 to C126, C118 to C127, C119 to C128, C120 to C129, C121 to C130, C122 to C131, C123 to C132, C124 to C133, C125 to C134, C126 to C135, C127 to C136
