File: test_boards/3CH-AWG-TIA/tfl.kicad_sch (KiCad schematic)
At the start: 7 parts, among them U9 LM311

Commit message: Добавлен anchor_role в генерируемые шаблоны
Parts:
- renumbered D12 to D13, R45 to R46, R46 to R47, R47 to R48

Commit message: Теперь можно использовать  anchor_role, anchor_cluster в thermal_via_array и manual positions
Parts:
- renumbered C128 to C137, C129 to C138
Changed lines of the file:
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@@
 		(dnp no)
 		(fields_autoplaced yes)
-		(property "Reference" "C128"
+		(property "Reference" "C137"
 			(at 55.88 50.7999 0)
 			(show_name no)
@@
 			(project "3CH-AWG-TIA"
 				(path "/1e22769e-c24b-4bb1-9c9f-ec579d192217/37fadcfc-2053-465b-a57f-61f3ae87f57a/5aaff5b5-4f08-4c6b-b668-79f4c527a860"
-					(reference "C162")
-					(unit 1)
-				)
-				(path "/1e22769e-c24b-4bb1-9c9f-ec579d192217/6b018f07-dde5-4cc8-ba46-360bc68cf3d3/5aaff5b5-4f08-4c6b-b668-79f4c527a860"
-					(reference "C196")
-					(unit 1)
-				)
-				(path "/1e22769e-c24b-4bb1-9c9f-ec579d192217/fb16a0a4-f706-49de-9d7e-e9bca2583031/5aaff5b5-4f08-4c6b-b668-79f4c527a860"
-					(reference "C128")
+					(reference "C171")
+					(unit 1)
+				)
+				(path "/1e22769e-c24b-4bb1-9c9f-ec579d192217/6b018f07-dde5-4cc8-ba46-360bc68cf3d3/5aaff5b5-4f08-4c6b-b668-79f4c527a860"
+					(reference "C205")
+					(unit 1)
+				)
+				(path "/1e22769e-c24b-4bb1-9c9f-ec579d192217/fb16a0a4-f706-49de-9d7e-e9bca2583031/5aaff5b5-4f08-4c6b-b668-79f4c527a860"
+					(reference "C137")
 					(unit 1)
 				)
@@
 		(dnp no)
 		(fields_autoplaced yes)
-		(property "Reference" "C129"
+		(property "Reference" "C138"
 			(at 67.31 50.7999 0)
 			(show_name no)
@@
 			(project "3CH-AWG-TIA"
 				(path "/1e22769e-c24b-4bb1-9c9f-ec579d192217/37fadcfc-2053-465b-a57f-61f3ae87f57a/5aaff5b5-4f08-4c6b-b668-79f4c527a860"
-					(reference "C163")
-					(unit 1)
-				)
-				(path "/1e22769e-c24b-4bb1-9c9f-ec579d192217/6b018f07-dde5-4cc8-ba46-360bc68cf3d3/5aaff5b5-4f08-4c6b-b668-79f4c527a860"
-					(reference "C197")
-					(unit 1)
-				)
-				(path "/1e22769e-c24b-4bb1-9c9f-ec579d192217/fb16a0a4-f706-49de-9d7e-e9bca2583031/5aaff5b5-4f08-4c6b-b668-79f4c527a860"
-					(reference "C129")
-					(unit 1)
-				)
+					(reference "C172")
+					(unit 1)
+				)
+				(path "/1e22769e-c24b-4bb1-9c9f-ec579d192217/6b018f07-dde5-4cc8-ba46-360bc68cf3d3/5aaff5b5-4f08-4c6b-b668-79f4c527a860"
+					(reference "C206")
+					(unit 1)
+				)
+				(path "/1e22769e-c24b-4bb1-9c9f-ec579d192217/fb16a0a4-f706-49de-9d7e-e9bca2583031/5aaff5b5-4f08-4c6b-b668-79f4c527a860"
+					(reference "C138")
+					(unit 1)
+				)
