File: test_boards/3CH-AWG-TIA/fpga.kicad_sch (KiCad schematic)
At the start: 95 parts, among them IC1 10CL006YE144C8G, J3 CL_JTAG, U5 W25Q128JVS, Y1 SG-7050CAN

Commit message: Добавлен anchor_role в генерируемые шаблоны
Parts:
- C31, C45, C76, C82, FB7: Cluster (none) -> Pi_Filter_1V2_VCCINT
- C32, C46, C77, C83, FB8: Cluster (none) -> Pi_Filter_1V2_VCCD_PLL
- C33, C47, C78, C84, FB9: Cluster (none) -> Pi_Filter_1V2_VCCA_P2V5
- C34, C48, C79, C85, FB10: Cluster (none) -> Pi_Filter_3V3_VCCIO
- C88, C89, C90, C92: Cluster (none) -> R_Filter_3V3_Osc
- C91, C93, C94, C95: Cluster (none) -> Pi_Filter_3V3_Flash
- R15: renamed from R14; Cluster (none) -> R_Filter_3V3_Osc
- R18: renamed from R17; Cluster (none) -> Channel_0_Signal_Matcher
- R19: renamed from R18; Cluster (none) -> Channel_0_Signal_Matcher
- R20: renamed from R19; Cluster (none) -> Channel_1_Signal_Matcher
- R21: renamed from R20; Cluster (none) -> Channel_1_Signal_Matcher
- R22: renamed from R21; Cluster (none) -> Channel_2_Signal_Matcher
- R23: renamed from R22; Cluster (none) -> Channel_2_Signal_Matcher
- R24: renamed from R23; Cluster (none) -> Pi_Filter_3V3_Flash
- renumbered R10 to R11, R11 to R12, R12 to R13, R13 to R14, R15 to R16, R16 to R17, R24 to R25, R25 to R26, R26 to R27, R27 to R28, R28 to R29, R29 to R30, R30 to R31, R31 to R32

Commit message: Теперь можно использовать  anchor_role, anchor_cluster в thermal_via_array и manual positions
Parts:
- added C45, C46: 100 nF, Capacitor_SMD:C_0402_1005Metric_Pad0.74x0.62mm_HandSolder, symbol Device:C
- added C58, C59, C60, C61, C62, C79, C80: 4.7 uF, Capacitor_SMD:C_0603_1608Metric_Pad1.08x0.95mm_HandSolder, symbol Device:C
- C35, C36, C37, C38, C39, C40, C41, C42, C43, C44: Cluster (none) -> VCCIO_BANK
- C51: renamed from C60; Cluster (none) -> VCCIO_BANK
- C52: renamed from C61; Cluster (none) -> VCCIO_BANK
- C53: renamed from C62; Cluster (none) -> VCCIO_BANK
- C54: renamed from C63; Cluster (none) -> VCCIO_BANK
- C55: renamed from C64; Cluster (none) -> VCCIO_BANK
- C56: renamed from C65; Cluster (none) -> VCCIO_BANK
- C57: renamed from C66; Cluster (none) -> VCCIO_BANK
- C63: renamed from C49; Cluster (none) -> VCCINT_BANK
- C64: renamed from C50; Cluster (none) -> VCCINT_BANK
- C65: renamed from C51; Cluster (none) -> VCCINT_BANK
- C66: renamed from C52; Cluster (none) -> VCCINT_BANK
- C67: renamed from C53; Cluster (none) -> VCCINT_BANK
- C68: renamed from C54; Cluster (none) -> VCCINT_BANK
- C69: renamed from C55; Cluster (none) -> VCCINT_BANK
- C70: renamed from C56; Cluster (none) -> VCCINT_BANK
- C71: renamed from C57; Cluster (none) -> VCCINT_BANK
- C72: renamed from C69; Cluster (none) -> VCCINT_BANK
- C73: renamed from C70; Cluster (none) -> VCCINT_BANK
- C74: renamed from C71; Cluster (none) -> VCCINT_BANK
- C75: renamed from C72; Cluster (none) -> VCCINT_BANK
- C76: renamed from C73; Cluster (none) -> VCCINT_BANK
- C77: renamed from C74; Cluster (none) -> VCCINT_BANK
- C78: renamed from C75; Cluster (none) -> VCCINT_BANK
- C85: renamed from C86; Cluster (none) -> PLL_BANK
- C86: renamed from C87; Cluster (none) -> PLL_BANK
- C87: renamed from C80; Cluster (none) -> VCCA_BANK
- C88: renamed from C81; Cluster (none) -> VCCA_BANK
- C93: renamed from C67; Cluster (none) -> PLL_BANK
- C94: renamed from C68; Cluster (none) -> PLL_BANK
- C95: renamed from C58; Cluster (none) -> VCCA_BANK
- C96: renamed from C59; Cluster (none) -> VCCA_BANK
- Y1: Role OSC -> OSC_FPGA
- renumbered C91 to C100, C92 to C101, C93 to C102, C94 to C103, C95 to C104, C45 to C47, C46 to C48, C47 to C49, C48 to C50, C76 to C81, C77 to C82, C78 to C83, C79 to C84, C82 to C89, C83 to C90, C84 to C91, C85 to C92, C88 to C97, C89 to C98, C90 to C99
Connections:
- net +1V2_VCCINT: now also C79.1, C80.1
- net +3V3_VCCIO: now also C45.1, C46.1, C58.1, C59.1, C60.1, C61.1, C62.1
- net GND: now also C45.2, C46.2, C58.2, C59.2, C60.2, C61.2, C62.2, C79.2, C80.2
Other:
- moved on the sheet: C35, C36, C37, C38, C39, C40, C41, C42, C43, C44, C51, C52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

Commit message: Правки участков мёртвого кода и багов по тестам
Parts:
- C35, C36, C37, C38, C39, C40, C41, C42, C43, C44, C45, C46, C51, C52, C53, C54, C55, C56, C57, C58, C59, C60, C61, C62: Cluster VCCIO_BANK -> FPGA_PWR_BANK
- C63, C64, C65, C66, C67, C68, C69, C70, C71, C72, C73, C74, C75, C76, C77, C78, C79, C80: Cluster VCCINT_BANK -> FPGA_PWR_BANK
- C85, C86, C93, C94: Cluster PLL_BANK -> FPGA_PWR_BANK
- C87, C88, C95, C96: Cluster VCCA_BANK -> FPGA_PWR_BANK
Changed lines of the file:
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@@
 			)
 		)
-		(property "Cluster" "VCCINT_BANK"
+		(property "Cluster" "FPGA_PWR_BANK"
 			(at 58.42 149.86 90)
 			(hide yes)
@@
 			)
 		)
-		(property "Cluster" "VCCIO_BANK"
+		(property "Cluster" "FPGA_PWR_BANK"
 			(at 29.21 161.29 0)
 			(hide yes)
@@
 			)
 		)
-		(property "Cluster" "VCCIO_BANK"
+		(property "Cluster" "FPGA_PWR_BANK"
 			(at 41.91 264.16 90)
 			(hide yes)
@@
 			)
 		)
-		(property "Cluster" "VCCIO_BANK"
+		(property "Cluster" "FPGA_PWR_BANK"
 			(at -212.09 283.21 0)
 			(hide yes)
@@
 			)
 		)
-		(property "Cluster" "VCCINT_BANK"
+		(property "Cluster" "FPGA_PWR_BANK"
 			(at 72.39 218.44 90)
 			(hide yes)
@@
 			)
 		)
-		(property "Cluster" "VCCA_BANK"
+		(property "Cluster" "FPGA_PWR_BANK"
 			(at 87.63 185.42 0)
 			(hide yes)
@@
 			)
 		)
-		(property "Cluster" "VCCINT_BANK"
+		(property "Cluster" "FPGA_PWR_BANK"
 			(at 58.42 207.01 90)
 			(hide yes)
@@
 			)
 		)
-		(property "Cluster" "VCCA_BANK"
+		(property "Cluster" "FPGA_PWR_BANK"
 			(at 104.14 185.42 0)
 			(hide yes)
@@
 			)
 		)
-		(property "Cluster" "VCCIO_BANK"
+		(property "Cluster" "FPGA_PWR_BANK"
 			(at -166.37 226.06 0)
 			(hide yes)
@@
 			)
 		)
-		(property "Cluster" "VCCIO_BANK"
+		(property "Cluster" "FPGA_PWR_BANK"
 			(at -212.09 271.78 0)
 			(hide yes)
@@
 			)
 		)
-		(property "Cluster" "VCCIO_BANK"
+		(property "Cluster" "FPGA_PWR_BANK"
 			(at -200.66 260.35 0)
 			(hide yes)
@@
 			)
 		)
-		(property "Cluster" "VCCIO_BANK"
+		(property "Cluster" "FPGA_PWR_BANK"
 			(at 41.91 218.44 90)
 			(hide yes)
@@
 			)
 		)
-		(property "Cluster" "VCCINT_BANK"
+		(property "Cluster" "FPGA_PWR_BANK"
 			(at 72.39 161.29 90)
 			(hide yes)
@@
 			)
 		)
-		(property "Cluster" "VCCINT_BANK"
+		(property "Cluster" "FPGA_PWR_BANK"
 			(at 72.39 195.58 90)
 			(hide yes)
@@
 			)
 		)
-		(property "Cluster" "VCCIO_BANK"
+		(property "Cluster" "FPGA_PWR_BANK"
 			(at -212.09 294.64 0)
 			(hide yes)
@@
 			)
 		)
-		(property "Cluster" "PLL_BANK"
+		(property "Cluster" "FPGA_PWR_BANK"
 			(at 87.63 138.43 0)
 			(hide yes)
@@
 			)
 		)
-		(property "Cluster" "VCCIO_BANK"
+		(property "Cluster" "FPGA_PWR_BANK"
 			(at 41.91 172.72 90)
 			(hide yes)
@@
 			)
 		)
-		(property "Cluster" "PLL_BANK"
+		(property "Cluster" "FPGA_PWR_BANK"
 			(at 104.14 151.13 0)
 			(hide yes)
@@
 			)
 		)
-		(property "Cluster" "VCCINT_BANK"
+		(property "Cluster" "FPGA_PWR_BANK"
 			(at 72.39 172.72 90)
 			(hide yes)
@@
 			)
 		)
-		(property "Cluster" "VCCIO_BANK"
+		(property "Cluster" "FPGA_PWR_BANK"
 			(at 41.91 252.73 90)
 			(hide yes)
@@
 			)
 		)
-		(property "Cluster" "VCCIO_BANK"
+		(property "Cluster" "FPGA_PWR_BANK"
 			(at 41.91 184.15 90)
 			(hide yes)
@@
 			)
 		)
-		(property "Cluster" "VCCIO_BANK"
+		(property "Cluster" "FPGA_PWR_BANK"
 			(at -177.8 237.49 0)
 			(hide yes)
@@
 			)
 		)
-		(property "Cluster" "VCCIO_BANK"
+		(property "Cluster" "FPGA_PWR_BANK"
 			(at 41.91 229.87 90)
 			(hide yes)
@@
 			)
 		)
-		(property "Cluster" "VCCIO_BANK"
+		(property "Cluster" "FPGA_PWR_BANK"
 			(at 41.91 149.86 90)
 			(hide yes)
@@
 			)
 		)
-		(property "Cluster" "VCCINT_BANK"
+		(property "Cluster" "FPGA_PWR_BANK"
 			(at 72.39 229.87 90)
 			(hide yes)
@@
 			)
 		)
-		(property "Cluster" "VCCINT_BANK"
+		(property "Cluster" "FPGA_PWR_BANK"
 			(at 72.39 138.43 90)
 			(hide yes)
@@
 			)
 		)
-		(property "Cluster" "VCCIO_BANK"
+		(property "Cluster" "FPGA_PWR_BANK"
 			(at 41.91 161.29 90)
 			(hide yes)
@@
 			)
 		)
-		(property "Cluster" "VCCINT_BANK"
+		(property "Cluster" "FPGA_PWR_BANK"
 			(at 72.39 184.15 90)
 			(hide yes)
@@
 			)
 		)
-		(property "Cluster" "VCCINT_BANK"
+		(property "Cluster" "FPGA_PWR_BANK"
 			(at 58.42 195.58 90)
 			(hide yes)
@@
 			)
 		)
-		(property "Cluster" "VCCIO_BANK"
+		(property "Cluster" "FPGA_PWR_BANK"
 			(at 41.91 207.01 90)
 			(hide yes)
@@
 			)
 		)
-		(property "Cluster" "VCCIO_BANK"
+		(property "Cluster" "FPGA_PWR_BANK"
 			(at 41.91 195.58 90)
 			(hide yes)
@@
 			)
 		)
-		(property "Cluster" "PLL_BANK"
+		(property "Cluster" "FPGA_PWR_BANK"
 			(at 104.14 139.7 0)
 			(hide yes)
@@
 			)
 		)
-		(property "Cluster" "VCCIO_BANK"
+		(property "Cluster" "FPGA_PWR_BANK"
 			(at -120.65 180.34 0)
 			(hide yes)
@@
 			)
 		)
-		(property "Cluster" "VCCIO_BANK"
+		(property "Cluster" "FPGA_PWR_BANK"
 			(at 41.91 241.3 90)
 			(hide yes)
@@
 			)
 		)
-		(property "Cluster" "VCCIO_BANK"
+		(property "Cluster" "FPGA_PWR_BANK"
 			(at -143.51 203.2 0)
 			(hide yes)
@@
 			)
 		)
-		(property "Cluster" "VCCINT_BANK"
+		(property "Cluster" "FPGA_PWR_BANK"
 			(at 58.42 172.72 90)
 			(hide yes)
@@
 			)
 		)
-		(property "Cluster" "VCCIO_BANK"
+		(property "Cluster" "FPGA_PWR_BANK"
 			(at 29.21 138.43 0)
 			(hide yes)
@@
 			)
 		)
-		(property "Cluster" "PLL_BANK"
+		(property "Cluster" "FPGA_PWR_BANK"
 			(at 87.63 149.86 0)
 			(hide yes)
@@
 			)
 		)
-		(property "Cluster" "VCCINT_BANK"
+		(property "Cluster" "FPGA_PWR_BANK"
 			(at 58.42 218.44 90)
 			(hide yes)
@@
 			)
 		)
-		(property "Cluster" "VCCIO_BANK"
+		(property "Cluster" "FPGA_PWR_BANK"
 			(at 41.91 138.43 90)
 			(hide yes)
@@
 			)
 		)
-		(property "Cluster" "VCCINT_BANK"
+		(property "Cluster" "FPGA_PWR_BANK"
 			(at 58.42 161.29 90)
 			(hide yes)
@@
 			)
 		)
-		(property "Cluster" "VCCINT_BANK"
+		(property "Cluster" "FPGA_PWR_BANK"
 			(at 72.39 207.01 90)
 			(hide yes)
@@
 			)
 		)
-		(property "Cluster" "VCCINT_BANK"
+		(property "Cluster" "FPGA_PWR_BANK"
 			(at 58.42 184.15 90)
 			(hide yes)
@@
 			)
 		)
-		(property "Cluster" "VCCIO_BANK"
+		(property "Cluster" "FPGA_PWR_BANK"
 			(at -154.94 214.63 0)
 			(hide yes)
@@
 			)
 		)
-		(property "Cluster" "VCCINT_BANK"
+		(property "Cluster" "FPGA_PWR_BANK"
 			(at 72.39 149.86 90)
 			(hide yes)
@@
 			)
 		)
-		(property "Cluster" "VCCIO_BANK"
+		(property "Cluster" "FPGA_PWR_BANK"
 			(at -189.23 248.92 0)
 			(hide yes)
@@
 			)
 		)
-		(property "Cluster" "VCCINT_BANK"
+		(property "Cluster" "FPGA_PWR_BANK"
 			(at 58.42 138.43 90)
 			(hide yes)
@@
 			)
 		)
-		(property "Cluster" "VCCA_BANK"
+		(property "Cluster" "FPGA_PWR_BANK"
 			(at 87.63 173.99 0)
 			(hide yes)
@@
 			)
 		)
-		(property "Cluster" "VCCINT_BANK"
+		(property "Cluster" "FPGA_PWR_BANK"
 			(at 58.42 229.87 90)
 			(hide yes)
@@
 			)
 		)
-		(property "Cluster" "VCCA_BANK"
+		(property "Cluster" "FPGA_PWR_BANK"
 			(at 104.14 173.99 0)
 			(hide yes)
