File: test_boards/3CH-AWG-TIA/3CH-AWG-TIA.kicad_pcb (KiCad board)
At the start: 4 copper layers, 232.8 x 114.7 mm, 353 parts, among them IC1 10CL006YE144C8G, IC2 AD9707BCPZ, IC3 AD9707BCPZ, IC4 AD9707BCPZ, J1 ±5V In, J2 +-18V_PA, J3 CL_JTAG, J4 Signal Out, J5 Signal Out, J6 Signal Out, U1 AMS1117-1.2, U10 ADA4807-2ARM, U11 PC817, U12 ADA4870ARRZ, U13 LM311, U14 ADA4807-2ARM, U15 PC817, U16 ADA4870ARRZ, U17 LM311, U2 AMS1117CD-3.3, U3 LM317_TO-252, U4 LM337_TO252, U5 W25Q128JVS, U6 ADA4807-2ARM, U7 PC817, U8 ADA4870ARRZ, U9 LM311, Y1 SG-7050CAN

Commit message: Теперь можно использовать  anchor_role, anchor_cluster в thermal_via_array и manual positions
Parts:
- added C198: 1 nF, Capacitor_SMD:C_0603_1608Metric_Pad1.08x0.95mm_HandSolder, F.Cu at (148.8, 36.5)
- added C199: 22uF, Capacitor_Tantalum_SMD:CP_EIA-7343-20_Kemet-V, F.Cu at (156.0, 38.2)
- added C200: 22uF, Capacitor_Tantalum_SMD:CP_EIA-7343-20_Kemet-V, F.Cu at (156.0, 44.0)
- added C201: 100nF, Capacitor_SMD:C_0603_1608Metric_Pad1.08x0.95mm_HandSolder, F.Cu at (148.8, 39.0)
- added C202: 100nF, Capacitor_SMD:C_0603_1608Metric_Pad1.08x0.95mm_HandSolder, F.Cu at (148.8, 41.5)
- added C203: 1.9 pF, Capacitor_SMD:C_0603_1608Metric_Pad1.08x0.95mm_HandSolder, F.Cu at (148.8, 44.0)
- added C204: 22 pF, Capacitor_SMD:C_0603_1608Metric_Pad1.08x0.95mm_HandSolder, F.Cu at (148.8, 46.5)
- added C205: 1uF, Capacitor_SMD:C_0603_1608Metric_Pad1.08x0.95mm_HandSolder, F.Cu at (148.8, 51.0)
- added C206: 100nF, Capacitor_SMD:C_0603_1608Metric_Pad1.08x0.95mm_HandSolder, F.Cu at (148.8, 53.6)
- added D19: BAT54S, Package_TO_SOT_SMD:SOT-23, F.Cu at (153.5, 52.0)
- added R80: 10K, Resistor_SMD:R_0603_1608Metric_Pad0.98x0.95mm_HandSolder, F.Cu at (148.8, 56.1)
- C101: footprint Capacitor_SMD:C_0603_1608Metric_Pad1.08x0.95mm_HandSolder -> Capacitor_SMD:C_0402_1005Metric_Pad0.74x0.62mm_HandSolder
- C108, C113, C142, C147, C176, C181, C90, C91, C94, C96, C98: value 1uF -> 100 nF; footprint Capacitor_SMD:C_0603_1608Metric_Pad1.08x0.95mm_HandSolder -> Capacitor_SMD:C_0402_1005Metric_Pad0.74x0.62mm_HandSolder
- C110, C144, C178: value 1uF -> 100 nF
- C112, C116, C146, C150, C180, C184, C82, C83, C84, C97, C99: value 100 nF -> 1uF; footprint Capacitor_SMD:C_0402_1005Metric_Pad0.74x0.62mm_HandSolder -> Capacitor_SMD:C_0603_1608Metric_Pad1.08x0.95mm_HandSolder
- C117, C118, C151, C152, C185, C186: value 470 uF -> 1uF; footprint Capacitor_THT:CP_Radial_D10.0mm_P5.00mm -> Capacitor_SMD:C_0603_1608Metric_Pad1.08x0.95mm_HandSolder
- C119, C153, C187: value 100nF -> 1uF
- C120, C124, C125, C154, C158, C159, C188, C192, C193: value 100nF -> 100 nF; footprint Capacitor_SMD:C_0603_1608Metric_Pad1.08x0.95mm_HandSolder -> Capacitor_SMD:C_0402_1005Metric_Pad0.74x0.62mm_HandSolder
- C121, C155, C189: value 1 nF -> 100 nF; footprint Capacitor_SMD:C_0603_1608Metric_Pad1.08x0.95mm_HandSolder -> Capacitor_SMD:C_0402_1005Metric_Pad0.74x0.62mm_HandSolder
- C122, C123, C156, C157, C190, C191: value 22uF -> 1uF; footprint Capacitor_Tantalum_SMD:CP_EIA-7343-20_Kemet-V -> Capacitor_SMD:C_0603_1608Metric_Pad1.08x0.95mm_HandSolder
- C126, C160, C194: value 1.9 pF -> 470 uF; footprint Capacitor_SMD:C_0603_1608Metric_Pad1.08x0.95mm_HandSolder -> Capacitor_THT:CP_Radial_D10.0mm_P5.00mm
- C127, C161, C195: value 22 pF -> 470 uF; footprint Capacitor_SMD:C_0603_1608Metric_Pad1.08x0.95mm_HandSolder -> Capacitor_THT:CP_Radial_D10.0mm_P5.00mm
- C128, C134, C162, C168, C196: value 1uF -> 100nF
- C130, C164: value 1uF -> 1 nF
- C131, C165: value 100 nF -> 22uF; footprint Capacitor_SMD:C_0402_1005Metric_Pad0.74x0.62mm_HandSolder -> Capacitor_Tantalum_SMD:CP_EIA-7343-20_Kemet-V
- C132, C166: value 1uF -> 22uF; footprint Capacitor_SMD:C_0603_1608Metric_Pad1.08x0.95mm_HandSolder -> Capacitor_Tantalum_SMD:CP_EIA-7343-20_Kemet-V
- C133, C138, C167, C172: value 100 nF -> 100nF; footprint Capacitor_SMD:C_0402_1005Metric_Pad0.74x0.62mm_HandSolder -> Capacitor_SMD:C_0603_1608Metric_Pad1.08x0.95mm_HandSolder
- C135, C169: value 100 nF -> 1.9 pF
- C136, C170: value 100 nF -> 22 pF; footprint Capacitor_SMD:C_0402_1005Metric_Pad0.74x0.62mm_HandSolder -> Capacitor_SMD:C_0603_1608Metric_Pad1.08x0.95mm_HandSolder
- C51, C52, C53, C54, C55, C56, C58, C59, C85: value 100 nF -> 4.7 uF; footprint Capacitor_SMD:C_0402_1005Metric_Pad0.74x0.62mm_HandSolder -> Capacitor_SMD:C_0603_1608Metric_Pad1.08x0.95mm_HandSolder
- C63, C64, C65, C66, C69, C70: value 4.7 uF -> 100 nF; footprint Capacitor_SMD:C_0603_1608Metric_Pad1.08x0.95mm_HandSolder -> Capacitor_SMD:C_0402_1005Metric_Pad0.74x0.62mm_HandSolder
- C76, C77, C78, C79, C88: value 1uF -> 4.7 uF
- C81: value 4.7 uF -> 1uF
- D10: value MBRS360BT3G -> LED; footprint Diode_SMD:D_SMC -> Diode_SMD:D_0805_2012Metric_Pad1.15x1.40mm_HandSolder
- D12, D15, D18: value BAT54S -> MBRS360BT3G; footprint Package_TO_SOT_SMD:SOT-23 -> Diode_SMD:D_SMC
- D13, D16: value MBRS360BT3G -> BAT54S; footprint Diode_SMD:D_SMC -> Package_TO_SOT_SMD:SOT-23
- D4: value D -> LED; footprint Diode_SMD:D_SMA_Handsoldering -> Diode_SMD:D_0805_2012Metric_Pad1.15x1.40mm_HandSolder
- D8: value LED -> D; footprint Diode_SMD:D_0805_2012Metric_Pad1.15x1.40mm_HandSolder -> Diode_SMD:D_SMA_Handsoldering
- R10: value 1K -> 220; footprint Resistor_SMD:R_0402_1005Metric_Pad0.72x0.64mm_HandSolder -> Resistor_SMD:R_0603_1608Metric_Pad0.98x0.95mm_HandSolder
- R11: value 10K -> 1K
- R12, R27: value 4.7K -> 10K
- R13: value 33 -> 4.7K
- R14, R23: value 2R2 -> 33
- R17: value 33 -> 2R2
- R24: value 10K -> 2R2
- R29: value 10K -> 4.7K
- R3: value 330 -> 50
- R32: value 22 -> 10K
- R34, R50, R66: value 8.2K -> 22
- R35, R51, R67: value 249 -> 8.2K
- R37, R53, R69: value 150R0 -> 249; footprint Resistor_SMD:R_0603_1608Metric_Pad0.98x0.95mm_HandSolder -> Resistor_SMD:R_0402_1005Metric_Pad0.72x0.64mm_HandSolder
- R38, R54, R70: value 140R0 -> 150R0
- R39, R55, R71: value 330 -> 140R0
- R4: value 240 -> 330
- R40, R56, R72: value 2K0 -> 330
- R41, R57, R73: value 10K0 -> 2K0
- R42, R58, R74: value 10K -> 10K0
- R43, R59, R75: value BPR56 22R -> 10K; footprint Resistor_THT:R_Axial_Power_L50.0mm_W9.0mm_P55.88mm -> Resistor_SMD:R_0603_1608Metric_Pad0.98x0.95mm_HandSolder
- R44, R60, R76: value 2K10 -> BPR56 22R; footprint Resistor_SMD:R_0603_1608Metric_Pad0.98x0.95mm_HandSolder -> Resistor_THT:R_Axial_Power_L50.0mm_W9.0mm_P55.88mm
- R45, R61, R77: value 560 -> 2K10; footprint Resistor_SMD:R_0402_1005Metric_Pad0.72x0.64mm_HandSolder -> Resistor_SMD:R_0603_1608Metric_Pad0.98x0.95mm_HandSolder
- R46, R62, R78: value 10K0 -> 560
- R47, R63, R79: value 10K -> 10K0; footprint Resistor_SMD:R_0603_1608Metric_Pad0.98x0.95mm_HandSolder -> Resistor_SMD:R_0402_1005Metric_Pad0.72x0.64mm_HandSolder
- R48, R64: value 22 -> 10K; footprint Resistor_SMD:R_0402_1005Metric_Pad0.72x0.64mm_HandSolder -> Resistor_SMD:R_0603_1608Metric_Pad0.98x0.95mm_HandSolder
- R8: value 220 -> 240
- moved IC1 272.9 mm to (59.4, 47.2)
Connections:
- C101 pad 1: /Channel_0/DAC/DAC_REFIO -> GND
- C101 pad 2: GND -> +3V3_OSCILL
- C103 pad 1: /Channel_0/DAC/+3V3_AVDD -> +3V3_FLASH
- C104 pad 1: /Channel_0/DAC/+3V3_AVDD -> GND
- C104 pad 2: GND -> +3V3_FLASH
- C107 pad 1: /Channel_0/DAC/+3V3_DVDD -> /Channel_0/DAC/+3V3_CLKVDD
- C108 pad 1: /Channel_0/DAC/+3V3_DVDD -> /Channel_0/DAC/+3V3_CLKVDD
- C109 pad 1: +2V5 -> +3V3
- C110 pad 1: -2V5 -> /Channel_0/DAC/DAC_REFIO
- C111 pad 1: +2V5 -> +3V3
- C112 pad 1: -2V5 -> /Channel_0/DAC/+3V3_AVDD
- C113 pad 1: /Channel_0/OpAmp/+2V5_OA -> /Channel_0/DAC/+3V3_AVDD
- C114 pad 1: /Channel_0/OpAmp/-2V5_OA -> +3V3
- C115 pad 1: /Channel_0/OpAmp/+2V5_OA -> +3V3
- C116 pad 1: /Channel_0/OpAmp/-2V5_OA -> /Channel_0/DAC/+3V3_DVDD
- C117 pad 1: +18V_IN -> /Channel_0/DAC/+3V3_DVDD
- C118 pad 1: -18V_IN -> +2V5
- C119 pad 1: +18V_IN -> -2V5
- C120 pad 1: -18V_IN -> +2V5
- C121 pad 1: /Channel_0/Power Amplifier Sheet/PA_ON -> -2V5
- C121 pad 2: /Channel_0/Power Amplifier Sheet/-18V_PA -> GND
- C122 pad 1: /Channel_0/Power Amplifier Sheet/+18V_PA -> /Channel_0/OpAmp/+2V5_OA
- C123 pad 1: /Channel_0/Power Amplifier Sheet/-18V_PA -> /Channel_0/OpAmp/-2V5_OA
- C124 pad 1: /Channel_0/Power Amplifier Sheet/+18V_PA -> /Channel_0/OpAmp/+2V5_OA
- C125 pad 1: /Channel_0/Power Amplifier Sheet/-18V_PA -> /Channel_0/OpAmp/-2V5_OA
- C126 pad 1: /Channel_0/Power Amplifier Sheet/PA_IN_N -> +18V_IN
- C126 pad 2: /Channel_0/Power Amplifier Sheet/PA_SIGNAL -> GND
- C127 pad 1: /Channel_0/Power Amplifier Sheet/PA_SIGNAL_OUT -> -18V_IN
- C128 pad 1: +3V3 -> +18V_IN
- C129 pad 1: +3V3 -> -18V_IN
- C130 pad 1: +3V3 -> /Channel_0/Power Amplifier Sheet/PA_ON
- C130 pad 2: GND -> /Channel_0/Power Amplifier Sheet/-18V_PA
- C131 pad 1: +3V3 -> /Channel_0/Power Amplifier Sheet/+18V_PA
- C132 pad 1: /Channel_1/DAC/+3V3_CLKVDD -> /Channel_0/Power Amplifier Sheet/-18V_PA
- C133 pad 1: /Channel_1/DAC/+3V3_CLKVDD -> /Channel_0/Power Amplifier Sheet/+18V_PA
- C134 pad 1: +3V3 -> /Channel_0/Power Amplifier Sheet/-18V_PA
- C135 pad 1: /Channel_1/DAC/DAC_REFIO -> /Channel_0/Power Amplifier Sheet/PA_IN_N
- C135 pad 2: GND -> /Channel_0/Power Amplifier Sheet/PA_SIGNAL
- C136 pad 1: +3V3 -> /Channel_0/Power Amplifier Sheet/PA_SIGNAL_OUT
- C137 pad 1: /Channel_1/DAC/+3V3_AVDD -> +3V3
- C138 pad 1: /Channel_1/DAC/+3V3_AVDD -> +3V3
- C141 pad 1: /Channel_1/DAC/+3V3_DVDD -> /Channel_1/DAC/+3V3_CLKVDD
- C142 pad 1: /Channel_1/DAC/+3V3_DVDD -> /Channel_1/DAC/+3V3_CLKVDD
- C143 pad 1: +2V5 -> +3V3
- C144 pad 1: -2V5 -> /Channel_1/DAC/DAC_REFIO
- C145 pad 1: +2V5 -> +3V3
- C146 pad 1: -2V5 -> /Channel_1/DAC/+3V3_AVDD
- C147 pad 1: /Channel_1/OpAmp/+2V5_OA -> /Channel_1/DAC/+3V3_AVDD
- C148 pad 1: /Channel_1/OpAmp/-2V5_OA -> +3V3
- C149 pad 1: /Channel_1/OpAmp/+2V5_OA -> +3V3
- C150 pad 1: /Channel_1/OpAmp/-2V5_OA -> /Channel_1/DAC/+3V3_DVDD
- C151 pad 1: +18V_IN -> /Channel_1/DAC/+3V3_DVDD
- C152 pad 1: -18V_IN -> +2V5
- C153 pad 1: +18V_IN -> -2V5
- C154 pad 1: -18V_IN -> +2V5
- C155 pad 1: /Channel_1/Power Amplifier Sheet/PA_ON -> -2V5
- C155 pad 2: /Channel_1/Power Amplifier Sheet/-18V_PA -> GND
- C156 pad 1: /Channel_1/Power Amplifier Sheet/+18V_PA -> /Channel_1/OpAmp/+2V5_OA
- C157 pad 1: /Channel_1/Power Amplifier Sheet/-18V_PA -> /Channel_1/OpAmp/-2V5_OA
- C158 pad 1: /Channel_1/Power Amplifier Sheet/+18V_PA -> /Channel_1/OpAmp/+2V5_OA
- C159 pad 1: /Channel_1/Power Amplifier Sheet/-18V_PA -> /Channel_1/OpAmp/-2V5_OA
- C160 pad 1: /Channel_1/Power Amplifier Sheet/PA_IN_N -> +18V_IN
- C160 pad 2: /Channel_1/Power Amplifier Sheet/PA_SIGNAL -> GND
- C161 pad 1: /Channel_1/Power Amplifier Sheet/PA_SIGNAL_OUT -> -18V_IN
- C162 pad 1: +3V3 -> +18V_IN
- C163 pad 1: +3V3 -> -18V_IN
- C164 pad 1: +3V3 -> /Channel_1/Power Amplifier Sheet/PA_ON
- C164 pad 2: GND -> /Channel_1/Power Amplifier Sheet/-18V_PA
- C165 pad 1: +3V3 -> /Channel_1/Power Amplifier Sheet/+18V_PA
- C166 pad 1: /Channel_2/DAC/+3V3_CLKVDD -> /Channel_1/Power Amplifier Sheet/-18V_PA
- C167 pad 1: /Channel_2/DAC/+3V3_CLKVDD -> /Channel_1/Power Amplifier Sheet/+18V_PA
- C168 pad 1: +3V3 -> /Channel_1/Power Amplifier Sheet/-18V_PA
- C169 pad 1: /Channel_2/DAC/DAC_REFIO -> /Channel_1/Power Amplifier Sheet/PA_IN_N
- C169 pad 2: GND -> /Channel_1/Power Amplifier Sheet/PA_SIGNAL
- C170 pad 1: +3V3 -> /Channel_1/Power Amplifier Sheet/PA_SIGNAL_OUT
- C171 pad 1: /Channel_2/DAC/+3V3_AVDD -> +3V3
- C172 pad 1: /Channel_2/DAC/+3V3_AVDD -> +3V3
- C175 pad 1: /Channel_2/DAC/+3V3_DVDD -> /Channel_2/DAC/+3V3_CLKVDD
- C176 pad 1: /Channel_2/DAC/+3V3_DVDD -> /Channel_2/DAC/+3V3_CLKVDD
- C177 pad 1: +2V5 -> +3V3
- C178 pad 1: -2V5 -> /Channel_2/DAC/DAC_REFIO
- C179 pad 1: +2V5 -> +3V3
- C180 pad 1: -2V5 -> /Channel_2/DAC/+3V3_AVDD
- C181 pad 1: /Channel_2/OpAmp/+2V5_OA -> /Channel_2/DAC/+3V3_AVDD
- C182 pad 1: /Channel_2/OpAmp/-2V5_OA -> +3V3
- C183 pad 1: /Channel_2/OpAmp/+2V5_OA -> +3V3
- C184 pad 1: /Channel_2/OpAmp/-2V5_OA -> /Channel_2/DAC/+3V3_DVDD
- C185 pad 1: +18V_IN -> /Channel_2/DAC/+3V3_DVDD
- C186 pad 1: -18V_IN -> +2V5
- C187 pad 1: +18V_IN -> -2V5
- C188 pad 1: -18V_IN -> +2V5
- C189 pad 1: /Channel_2/Power Amplifier Sheet/PA_ON -> -2V5
- C189 pad 2: /Channel_2/Power Amplifier Sheet/-18V_PA -> GND
- C190 pad 1: /Channel_2/Power Amplifier Sheet/+18V_PA -> /Channel_2/OpAmp/+2V5_OA
- C191 pad 1: /Channel_2/Power Amplifier Sheet/-18V_PA -> /Channel_2/OpAmp/-2V5_OA
- C192 pad 1: /Channel_2/Power Amplifier Sheet/+18V_PA -> /Channel_2/OpAmp/+2V5_OA
- C193 pad 1: /Channel_2/Power Amplifier Sheet/-18V_PA -> /Channel_2/OpAmp/-2V5_OA
- C194 pad 1: /Channel_2/Power Amplifier Sheet/PA_IN_N -> +18V_IN
- C194 pad 2: /Channel_2/Power Amplifier Sheet/PA_SIGNAL -> GND
- C195 pad 1: /Channel_2/Power Amplifier Sheet/PA_SIGNAL_OUT -> -18V_IN
- C196 pad 1: +3V3 -> +18V_IN
- C197 pad 1: +3V3 -> -18V_IN
- C45 pad 1: +1V2 -> +3V3_VCCIO
- C46 pad 1: +1V2 -> +3V3_VCCIO
- C47 pad 1: +2V5 -> +1V2
- C48 pad 1: +3V3 -> +1V2
- C49 pad 1: +1V2_VCCINT -> +2V5
- C50 pad 1: +1V2_VCCINT -> +3V3
- C51 pad 1: +1V2_VCCINT -> +3V3_VCCIO
- C52 pad 1: +1V2_VCCINT -> +3V3_VCCIO
- C53 pad 1: +1V2_VCCINT -> +3V3_VCCIO
- C54 pad 1: +1V2_VCCINT -> +3V3_VCCIO
- C55 pad 1: +1V2_VCCINT -> +3V3_VCCIO
- C56 pad 1: +1V2_VCCINT -> +3V3_VCCIO
- C57 pad 1: +1V2_VCCINT -> +3V3_VCCIO
- C58 pad 1: +2V5_VCCA -> +3V3_VCCIO
- C59 pad 1: +2V5_VCCA -> +3V3_VCCIO
- C63 pad 1: +3V3_VCCIO -> +1V2_VCCINT
- C64 pad 1: +3V3_VCCIO -> +1V2_VCCINT
- C65 pad 1: +3V3_VCCIO -> +1V2_VCCINT
- C66 pad 1: +3V3_VCCIO -> +1V2_VCCINT
- C67 pad 1: +1V2_VCCD_PLL -> +1V2_VCCINT
- C68 pad 1: +1V2_VCCD_PLL -> +1V2_VCCINT
- C77 pad 1: +1V2_VCCD_PLL -> +1V2_VCCINT
- C78 pad 1: +2V5_VCCA -> +1V2_VCCINT
- C79 pad 1: +3V3_VCCIO -> +1V2_VCCINT
- C80 pad 1: +2V5_VCCA -> +1V2_VCCINT
- C81 pad 1: +2V5_VCCA -> +1V2_VCCINT
- C82 pad 1: +1V2_VCCINT -> +1V2_VCCD_PLL
- C83 pad 1: +1V2_VCCD_PLL -> +2V5_VCCA
- C84 pad 1: +2V5_VCCA -> +3V3_VCCIO
- C85 pad 1: +3V3_VCCIO -> +1V2_VCCD_PLL
- C87 pad 1: +1V2_VCCD_PLL -> +2V5_VCCA
- C88 pad 1: +3V3 -> +2V5_VCCA
- C89 pad 1: +3V3 -> +1V2_VCCINT
- C90 pad 1: +3V3_OSCILL -> +1V2_VCCD_PLL
- C91 pad 1: +3V3 -> +2V5_VCCA
- C92 pad 1: GND -> +3V3_VCCIO
- C92 pad 2: +3V3_OSCILL -> GND
- C93 pad 1: +3V3 -> +1V2_VCCD_PLL
- C94 pad 1: +3V3_FLASH -> +1V2_VCCD_PLL
- C95 pad 1: GND -> +2V5_VCCA
- C95 pad 2: +3V3_FLASH -> GND
- C96 pad 1: +3V3 -> +2V5_VCCA
- C98 pad 1: /Channel_0/DAC/+3V3_CLKVDD -> +3V3
- C99 pad 1: /Channel_0/DAC/+3V3_CLKVDD -> +3V3_OSCILL
- D10 pad 1: /Channel_0/Power Amplifier Sheet/+18V_PA -> GND
- D10 pad 2: /Channel_0/Power Amplifier Sheet/PA_SIGNAL -> /Power/+2V5_LED
- D11 pad 1: /Channel_0/Power Amplifier Sheet/PA_SIGNAL -> /Channel_0/Power Amplifier Sheet/+18V_PA
- D11 pad 2: /Channel_0/Power Amplifier Sheet/-18V_PA -> /Channel_0/Power Amplifier Sheet/PA_SIGNAL
- D12 pad 1: GND -> /Channel_0/Power Amplifier Sheet/PA_SIGNAL
- D12 pad 2: +3V3 -> /Channel_0/Power Amplifier Sheet/-18V_PA
- D13 pad 1: /Channel_1/Power Amplifier Sheet/+18V_PA -> GND
- D13 pad 2: /Channel_1/Power Amplifier Sheet/PA_SIGNAL -> +3V3
- D14 pad 1: /Channel_1/Power Amplifier Sheet/PA_SIGNAL -> /Channel_1/Power Amplifier Sheet/+18V_PA
- D14 pad 2: /Channel_1/Power Amplifier Sheet/-18V_PA -> /Channel_1/Power Amplifier Sheet/PA_SIGNAL
- D15 pad 1: GND -> /Channel_1/Power Amplifier Sheet/PA_SIGNAL
- D15 pad 2: +3V3 -> /Channel_1/Power Amplifier Sheet/-18V_PA
- D16 pad 1: /Channel_2/Power Amplifier Sheet/+18V_PA -> GND
- D16 pad 2: /Channel_2/Power Amplifier Sheet/PA_SIGNAL -> +3V3
- D17 pad 1: /Channel_2/Power Amplifier Sheet/PA_SIGNAL -> /Channel_2/Power Amplifier Sheet/+18V_PA
- D17 pad 2: /Channel_2/Power Amplifier Sheet/-18V_PA -> /Channel_2/Power Amplifier Sheet/PA_SIGNAL
- D18 pad 1: GND -> /Channel_2/Power Amplifier Sheet/PA_SIGNAL
- D18 pad 2: +3V3 -> /Channel_2/Power Amplifier Sheet/-18V_PA
- D3 pad 2: /Power/+3V3_LED -> /Power/+1V2_LED
- D4 pad 1: +5V -> GND
- D4 pad 2: +2V5_DIRTY -> /Power/+3V3_LED
- D5 pad 1: -5V -> +5V
- D5 pad 2: -2V5_DIRTY -> +2V5_DIRTY
- D6 pad 1: +2V5_DIRTY -> -5V
- D6 pad 2: /Power/+2V5_ADJ -> -2V5_DIRTY
- D7 pad 1: -2V5_DIRTY -> +2V5_DIRTY
- D7 pad 2: /Power/-2V5_ADJ -> /Power/+2V5_ADJ
- D8 pad 1: GND -> -2V5_DIRTY
- D8 pad 2: /Power/-2V5_LED -> /Power/-2V5_ADJ
- D9 pad 2: /Power/+2V5_LED -> /Power/-2V5_LED
- R10 pad 1: +3V3_OSCILL -> /Power/+2V5_LED
- R10 pad 2: /FPGA/CL_CLK_ON -> +2V5
- R11 pad 1: DAC_SPI_RESET -> +3V3_OSCILL
- R11 pad 2: GND -> /FPGA/CL_CLK_ON
- R12 pad 1: /FPGA/CL_TCK -> DAC_SPI_RESET
- R13 pad 1: /FPGA/CL_CLK_0 -> /FPGA/CL_TCK
- R13 pad 2: /FPGA/CL_CLK_0_IN -> GND
- R14 pad 1: +3V3 -> /FPGA/CL_CLK_0
- R14 pad 2: +3V3_OSCILL -> /FPGA/CL_CLK_0_IN
- R15 pad 1: /FPGA/FL_HOLD -> +3V3
- R15 pad 2: +3V3_FLASH -> +3V3_OSCILL
- R16 pad 1: /FPGA/FL_WP -> /FPGA/FL_HOLD
- R17 pad 1: /FPGA/DAC0_CLK_OUT_P -> /FPGA/FL_WP
- R17 pad 2: /Channel_0/DAC_CLK_P -> +3V3_FLASH
- R18 pad 1: /FPGA/DAC0_CLK_OUT_N -> /FPGA/DAC0_CLK_OUT_P
- R18 pad 2: /Channel_0/DAC_CLK_N -> /Channel_0/DAC_CLK_P
- R19 pad 1: /FPGA/DAC1_CLK_OUT_P -> /FPGA/DAC0_CLK_OUT_N
- R19 pad 2: /Channel_1/DAC_CLK_P -> /Channel_0/DAC_CLK_N
- R20 pad 1: /FPGA/DAC1_CLK_OUT_N -> /FPGA/DAC1_CLK_OUT_P
- R20 pad 2: /Channel_1/DAC_CLK_N -> /Channel_1/DAC_CLK_P
- R21 pad 1: /FPGA/DAC2_CLK_OUT_P -> /FPGA/DAC1_CLK_OUT_N
- R21 pad 2: /Channel_2/DAC_CLK_P -> /Channel_1/DAC_CLK_N
- R22 pad 1: /FPGA/DAC2_CLK_OUT_N -> /FPGA/DAC2_CLK_OUT_P
- R22 pad 2: /Channel_2/DAC_CLK_N -> /Channel_2/DAC_CLK_P
- R23 pad 1: +3V3 -> /FPGA/DAC2_CLK_OUT_N
- R23 pad 2: +3V3_FLASH -> /Channel_2/DAC_CLK_N
- R24 pad 1: /FPGA/CL_CONFIG_DONE -> +3V3
- R24 pad 2: +3V3_VCCIO -> +3V3_FLASH
- R25 pad 1: /FPGA/CL_NSTATUS -> /FPGA/CL_CONFIG_DONE
- R26 pad 1: /FPGA/CL_NCONFIG -> /FPGA/CL_NSTATUS
- R27 pad 1: /FPGA/CL_TMS -> /FPGA/CL_NCONFIG
- R28 pad 1: /FPGA/CL_TDI -> /FPGA/CL_TMS
- R29 pad 1: /FPGA/DAC0_SPI_CS -> /FPGA/CL_TDI
- R3 pad 1: /Power/+3V3_LED -> /Power/+1V2_LED
- R3 pad 2: +3V3 -> +1V2
- R30 pad 1: /FPGA/DAC1_SPI_CS -> /FPGA/DAC0_SPI_CS
- R31 pad 1: /FPGA/DAC2_SPI_CS -> /FPGA/DAC1_SPI_CS
- R32 pad 1: /Channel_0/DAC/DAC_OUT_P -> /FPGA/DAC2_SPI_CS
- R32 pad 2: /Channel_0/OpAmp/OA_IN_P -> +3V3_VCCIO
- R33 pad 1: /Channel_0/DAC/DAC_OUT_N -> /Channel_0/DAC/DAC_OUT_P
- R33 pad 2: /Channel_0/OpAmp/OA_IN_N -> /Channel_0/OpAmp/OA_IN_P
- R34 pad 1: /Channel_0/DAC/DAC_FS_ADJ -> /Channel_0/DAC/DAC_OUT_N
- R34 pad 2: GND -> /Channel_0/OpAmp/OA_IN_N
- R35 pad 1: /Channel_0/OpAmp/OA_IN_P -> /Channel_0/DAC/DAC_FS_ADJ
- R35 pad 2: /Channel_0/OpAmp/OA_OUT_P -> GND
- R36 pad 1: /Channel_0/OpAmp/OA_IN_N -> /Channel_0/OpAmp/OA_IN_P
- R36 pad 2: /Channel_0/OpAmp/OA_OUT_N -> /Channel_0/OpAmp/OA_OUT_P
- R37 pad 1: /Channel_0/OpAmp/OA_OUT_N -> /Channel_0/OpAmp/OA_IN_N
- R37 pad 2: /Channel_0/Power Amplifier Sheet/PA_IN_N -> /Channel_0/OpAmp/OA_OUT_N
- R38 pad 1: /Channel_0/OpAmp/OA_OUT_P -> /Channel_0/OpAmp/OA_OUT_N
- R38 pad 2: /Channel_0/OpAmp/PA_IN_P -> /Channel_0/Power Amplifier Sheet/PA_IN_N
- R39 pad 1: /Channel_0/Power Amplifier Sheet/PA_EN_IN -> /Channel_0/OpAmp/OA_OUT_P
- R39 pad 2: /Channel_0/PA_EN -> /Channel_0/OpAmp/PA_IN_P
- R4 pad 1: /Power/+2V5_ADJ -> /Power/+3V3_LED
- R4 pad 2: GND -> +3V3
- R40 pad 1: /Channel_0/Power Amplifier Sheet/-18V_PA -> /Channel_0/Power Amplifier Sheet/PA_EN_IN
- R40 pad 2: /Channel_0/Power Amplifier Sheet/PA_SD -> /Channel_0/PA_EN
- R41 pad 1: /Channel_0/Power Amplifier Sheet/PA_SD -> /Channel_0/Power Amplifier Sheet/-18V_PA
- R41 pad 2: GND -> /Channel_0/Power Amplifier Sheet/PA_SD
- R42 pad 2: /Channel_0/Power Amplifier Sheet/PA_ON -> GND
- R43 pad 1: /Channel_0/Power Amplifier Sheet/PA_SIGNAL -> /Channel_0/Power Amplifier Sheet/PA_SD
- R43 pad 2: /Channel_0/Power Amplifier Sheet/PA_SIGNAL_OUT -> /Channel_0/Power Amplifier Sheet/PA_ON
- R44 pad 1: /Channel_0/Power Amplifier Sheet/PA_IN_N -> /Channel_0/Power Amplifier Sheet/PA_SIGNAL
- R44 pad 2: /Channel_0/Power Amplifier Sheet/PA_SIGNAL -> /Channel_0/Power Amplifier Sheet/PA_SIGNAL_OUT
- R45 pad 1: /Channel_0/TFL/PA_TFL_V_REF -> /Channel_0/Power Amplifier Sheet/PA_IN_N
- R45 pad 2: /Channel_0/Power Amplifier Sheet/-18V_PA -> /Channel_0/Power Amplifier Sheet/PA_SIGNAL
- R46 pad 1: GND -> /Channel_0/TFL/PA_TFL_V_REF
- R46 pad 2: /Channel_0/TFL/PA_TFL_V_REF -> /Channel_0/Power Amplifier Sheet/-18V_PA
- R47 pad 1: +3V3 -> GND
- R47 pad 2: /Channel_0/TFL/CL_TFL_SIGNAL -> /Channel_0/TFL/PA_TFL_V_REF
- R48 pad 1: /Channel_1/DAC/DAC_OUT_P -> +3V3
- R48 pad 2: /Channel_1/OpAmp/OA_IN_P -> /Channel_0/TFL/CL_TFL_SIGNAL
- R49 pad 1: /Channel_1/DAC/DAC_OUT_N -> /Channel_1/DAC/DAC_OUT_P
- R49 pad 2: /Channel_1/OpAmp/OA_IN_N -> /Channel_1/OpAmp/OA_IN_P
- R5 pad 1: GND -> /Power/+2V5_ADJ
- R5 pad 2: /Power/-2V5_ADJ -> GND
- R50 pad 1: /Channel_1/DAC/DAC_FS_ADJ -> /Channel_1/DAC/DAC_OUT_N
- R50 pad 2: GND -> /Channel_1/OpAmp/OA_IN_N
- R51 pad 1: /Channel_1/OpAmp/OA_IN_P -> /Channel_1/DAC/DAC_FS_ADJ
- R51 pad 2: /Channel_1/OpAmp/OA_OUT_P -> GND
- R52 pad 1: /Channel_1/OpAmp/OA_IN_N -> /Channel_1/OpAmp/OA_IN_P
- R52 pad 2: /Channel_1/OpAmp/OA_OUT_N -> /Channel_1/OpAmp/OA_OUT_P
- R53 pad 1: /Channel_1/OpAmp/OA_OUT_N -> /Channel_1/OpAmp/OA_IN_N
- R53 pad 2: /Channel_1/Power Amplifier Sheet/PA_IN_N -> /Channel_1/OpAmp/OA_OUT_N
- R54 pad 1: /Channel_1/OpAmp/OA_OUT_P -> /Channel_1/OpAmp/OA_OUT_N
- R54 pad 2: /Channel_1/OpAmp/PA_IN_P -> /Channel_1/Power Amplifier Sheet/PA_IN_N
- R55 pad 1: /Channel_1/Power Amplifier Sheet/PA_EN_IN -> /Channel_1/OpAmp/OA_OUT_P
- R55 pad 2: /Channel_1/PA_EN -> /Channel_1/OpAmp/PA_IN_P
- R56 pad 1: /Channel_1/Power Amplifier Sheet/-18V_PA -> /Channel_1/Power Amplifier Sheet/PA_EN_IN
- R56 pad 2: /Channel_1/Power Amplifier Sheet/PA_SD -> /Channel_1/PA_EN
- R57 pad 1: /Channel_1/Power Amplifier Sheet/PA_SD -> /Channel_1/Power Amplifier Sheet/-18V_PA
- R57 pad 2: GND -> /Channel_1/Power Amplifier Sheet/PA_SD
- R58 pad 2: /Channel_1/Power Amplifier Sheet/PA_ON -> GND
- R59 pad 1: /Channel_1/Power Amplifier Sheet/PA_SIGNAL -> /Channel_1/Power Amplifier Sheet/PA_SD
- R59 pad 2: /Channel_1/Power Amplifier Sheet/PA_SIGNAL_OUT -> /Channel_1/Power Amplifier Sheet/PA_ON
- R6 pad 1: +2V5_DIRTY -> GND
- R6 pad 2: /Power/+2V5_ADJ -> /Power/-2V5_ADJ
- R60 pad 1: /Channel_1/Power Amplifier Sheet/PA_IN_N -> /Channel_1/Power Amplifier Sheet/PA_SIGNAL
- R60 pad 2: /Channel_1/Power Amplifier Sheet/PA_SIGNAL -> /Channel_1/Power Amplifier Sheet/PA_SIGNAL_OUT
- R61 pad 1: /Channel_1/TFL/PA_TFL_V_REF -> /Channel_1/Power Amplifier Sheet/PA_IN_N
- R61 pad 2: /Channel_1/Power Amplifier Sheet/-18V_PA -> /Channel_1/Power Amplifier Sheet/PA_SIGNAL
- R62 pad 1: GND -> /Channel_1/TFL/PA_TFL_V_REF
- R62 pad 2: /Channel_1/TFL/PA_TFL_V_REF -> /Channel_1/Power Amplifier Sheet/-18V_PA
- R63 pad 1: +3V3 -> GND
- R63 pad 2: /Channel_1/TFL/CL_TFL_SIGNAL -> /Channel_1/TFL/PA_TFL_V_REF
- R64 pad 1: /Channel_2/DAC/DAC_OUT_P -> +3V3
- R64 pad 2: /Channel_2/OpAmp/OA_IN_P -> /Channel_1/TFL/CL_TFL_SIGNAL
- R65 pad 1: /Channel_2/DAC/DAC_OUT_N -> /Channel_2/DAC/DAC_OUT_P
- R65 pad 2: /Channel_2/OpAmp/OA_IN_N -> /Channel_2/OpAmp/OA_IN_P
- R66 pad 1: /Channel_2/DAC/DAC_FS_ADJ -> /Channel_2/DAC/DAC_OUT_N
- R66 pad 2: GND -> /Channel_2/OpAmp/OA_IN_N
- R67 pad 1: /Channel_2/OpAmp/OA_IN_P -> /Channel_2/DAC/DAC_FS_ADJ
- R67 pad 2: /Channel_2/OpAmp/OA_OUT_P -> GND
- R68 pad 1: /Channel_2/OpAmp/OA_IN_N -> /Channel_2/OpAmp/OA_IN_P
- R68 pad 2: /Channel_2/OpAmp/OA_OUT_N -> /Channel_2/OpAmp/OA_OUT_P
- R69 pad 1: /Channel_2/OpAmp/OA_OUT_N -> /Channel_2/OpAmp/OA_IN_N
- R69 pad 2: /Channel_2/Power Amplifier Sheet/PA_IN_N -> /Channel_2/OpAmp/OA_OUT_N
- R7 pad 1: /Power/-2V5_ADJ -> +2V5_DIRTY
- R7 pad 2: -2V5_DIRTY -> /Power/+2V5_ADJ
- R70 pad 1: /Channel_2/OpAmp/OA_OUT_P -> /Channel_2/OpAmp/OA_OUT_N
- R70 pad 2: /Channel_2/OpAmp/PA_IN_P -> /Channel_2/Power Amplifier Sheet/PA_IN_N
- R71 pad 1: /Channel_2/Power Amplifier Sheet/PA_EN_IN -> /Channel_2/OpAmp/OA_OUT_P
- R71 pad 2: /Channel_2/PA_EN -> /Channel_2/OpAmp/PA_IN_P
- R72 pad 1: /Channel_2/Power Amplifier Sheet/-18V_PA -> /Channel_2/Power Amplifier Sheet/PA_EN_IN
- R72 pad 2: /Channel_2/Power Amplifier Sheet/PA_SD -> /Channel_2/PA_EN
- R73 pad 1: /Channel_2/Power Amplifier Sheet/PA_SD -> /Channel_2/Power Amplifier Sheet/-18V_PA
- R73 pad 2: GND -> /Channel_2/Power Amplifier Sheet/PA_SD
- R74 pad 2: /Channel_2/Power Amplifier Sheet/PA_ON -> GND
- R75 pad 1: /Channel_2/Power Amplifier Sheet/PA_SIGNAL -> /Channel_2/Power Amplifier Sheet/PA_SD
- R75 pad 2: /Channel_2/Power Amplifier Sheet/PA_SIGNAL_OUT -> /Channel_2/Power Amplifier Sheet/PA_ON
- R76 pad 1: /Channel_2/Power Amplifier Sheet/PA_IN_N -> /Channel_2/Power Amplifier Sheet/PA_SIGNAL
- R76 pad 2: /Channel_2/Power Amplifier Sheet/PA_SIGNAL -> /Channel_2/Power Amplifier Sheet/PA_SIGNAL_OUT
- R77 pad 1: /Channel_2/TFL/PA_TFL_V_REF -> /Channel_2/Power Amplifier Sheet/PA_IN_N
- R77 pad 2: /Channel_2/Power Amplifier Sheet/-18V_PA -> /Channel_2/Power Amplifier Sheet/PA_SIGNAL
- R78 pad 1: GND -> /Channel_2/TFL/PA_TFL_V_REF
- R78 pad 2: /Channel_2/TFL/PA_TFL_V_REF -> /Channel_2/Power Amplifier Sheet/-18V_PA
- R79 pad 1: +3V3 -> GND
- R79 pad 2: /Channel_2/TFL/CL_TFL_SIGNAL -> /Channel_2/TFL/PA_TFL_V_REF
- R8 pad 1: /Power/-2V5_LED -> /Power/-2V5_ADJ
- R8 pad 2: -2V5 -> -2V5_DIRTY
- R9 pad 1: /Power/+2V5_LED -> /Power/-2V5_LED
- R9 pad 2: +2V5 -> -2V5

Commit message: Правки участков мёртвого кода и багов по тестам
Parts:
- C35, C36, C37, C38, C39, C40, C41, C42, C43, C44, C45, C46, C51, C52, C53, C54, C55, C56, C57, C58, C59, C60, C61, C62, C63, C64, C65, C66, C67, C68, C69, C70, C72, C73, C74, C75, C76, C77, C78, C79, C85, C86, C87, C88, C93, C94, C95, C96: moved to B.Cu
- moved C96 281.7 mm to (130.8, 58.3), turned to 180 degrees
- moved C87 251.8 mm to (108.3, 73.8), turned to 180 degrees
- moved C73 247.5 mm to (108.3, 71.3), turned to 180 degrees
- moved C72 243.3 mm to (108.3, 60.8), turned to 180 degrees
- moved C79 240.3 mm to (116.0, 53.8), turned to 90 degrees
- moved C64 240.1 mm to (111.3, 71.3)
- moved C63 239.9 mm to (111.3, 60.8)
- moved C74 237.9 mm to (118.3, 79.3), turned to -90 degrees
- moved C70 235.6 mm to (116.0, 56.8), turned to -90 degrees
- moved C62 234.1 mm to (113.8, 53.8), turned to 90 degrees
- moved C65 233.2 mm to (118.3, 76.3), turned to 90 degrees
- moved C94 233.2 mm to (127.3, 56.8), turned to -90 degrees
- moved C86 232.7 mm to (127.3, 53.8), turned to 90 degrees
- moved C78 231.2 mm to (125.0, 53.8), turned to 90 degrees
- moved C75 230.7 mm to (125.3, 79.3), turned to -90 degrees
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Routing:
- net +3V3_VCCIO: track 0.00 -> 95.3 mm, vias 0 -> 24
- net +1V2_VCCINT: track 0.00 -> 64.4 mm, vias 0 -> 16
- net GND: track 0.00 -> 59.3 mm, vias 0 -> 80
- net +1V2_VCCD_PLL: track 0.00 -> 16.6 mm, vias 0 -> 4
- net +2V5_VCCA: track 0.00 -> 15.5 mm, vias 0 -> 4

Commit message: Изменения в генерирующем скрипте
Parts:
- C35, C36, C37, C38, C39, C40, C41, C42, C43, C44, C45, C46, C51, C52, C53, C54, C55, C56, C57, C58, C59, C60, C61, C62, C63, C64, C65, C66, C67, C68, C69, C70, C72, C73, C74, C75, C76, C77, C78, C79, C85, C86, C87, C88, C93, C94, C95, C96: moved to F.Cu
- moved C35 58.4 mm to (168.2, 79.7), turned to 180 degrees
- moved C36 58.4 mm to (168.2, 82.3), turned to 180 degrees
- moved C37 58.4 mm to (173.0, 89.7)
- moved C39 58.4 mm to (180.0, 89.7)
- moved C53 58.4 mm to (173.0, 92.7)
- moved C54 58.4 mm to (177.7, 92.7)
- moved C55 58.4 mm to (180.0, 92.7)
- moved C56 58.4 mm to (184.7, 92.7)
- moved C63 58.4 mm to (168.2, 74.2), turned to 180 degrees
- moved C64 58.4 mm to (168.2, 84.7), turned to 180 degrees
- moved C74 58.4 mm to (175.2, 92.7)
- moved C75 58.4 mm to (182.2, 92.7)
- moved C85 58.4 mm to (170.7, 92.7)
- moved C95 58.4 mm to (168.2, 87.2), turned to 180 degrees
- moved C38 58.4 mm to (177.7, 89.7)
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Routing:
- net +3V3_VCCIO: track 95.3 -> 0.00 mm, vias 24 -> 0
- net +1V2_VCCINT: track 64.4 -> 0.00 mm, vias 16 -> 0
- net GND: track 59.3 -> 0.00 mm, vias 80 -> 0
- net +1V2_VCCD_PLL: track 16.6 -> 0.00 mm, vias 4 -> 0
- net +2V5_VCCA: track 15.5 -> 0.00 mm, vias 4 -> 0
